Commit message: Corrections

File: robospect_description/urdf/bases/robospect_base.urdf.xacro (robot description, xacro)
@@ -5,5 +5,4 @@
   <!-- Robot mechanical and motor parameters -->
   <xacro:property name="PI" value="3.1415926535897931"/>
-  <xacro:property name="wheel_width" value="0.175" />
   <!-- BASE FOOTPRINT -->
   <xacro:if value="${publish_bf}">
@@ -33,5 +32,5 @@
   <link name="base_link">
     <inertial>
-      <mass value="125.0" />
+      <mass value="50.0" />
       <origin xyz="0 0 0" />
       <inertia  ixx="1.391" ixy="0.004"  ixz="0.0"  iyy="6.853"  iyz="0.0"  izz="6.125" />

File: robospect_description/urdf/bases/robospect_crane.gazebo.xacro (robot description, xacro)
@@ -17,3 +17,33 @@
     <material>Gazebo/Green</material>
   </gazebo>
+  <gazebo reference="base_link">
+    <material>Gazebo/SkyBlue</material>
+  </gazebo>
+  <gazebo reference="first_link">
+    <material>Gazebo/Grey</material>
+  </gazebo>
+  <gazebo reference="second_link">
+    <material>Gazebo/SkyBlue</material>
+  </gazebo>
+  <gazebo reference="third_link">
+    <material>Gazebo/SkyBlue</material>
+  </gazebo>
+  <gazebo reference="fourth_link">
+    <material>Gazebo/SkyBlue</material>
+  </gazebo>
+  <gazebo reference="fifth_link">
+    <material>Gazebo/SkyBlue</material>
+  </gazebo>
+  <gazebo reference="sixth_link">
+    <material>Gazebo/SkyBlue</material>
+  </gazebo>
+  <gazebo reference="sixth_aux_link">
+    <material>Gazebo/SkyBlue</material>
+  </gazebo>
+  <gazebo reference="seventh_link">
+    <material>Gazebo/SkyBlue</material>
+  </gazebo>
+  <gazebo reference="tip_link">
+    <material>Gazebo/Grey</material>
+  </gazebo>
 </robot>

File: robospect_description/urdf/bases/robospect_crane.urdf.xacro (robot description, xacro)
@@ -1,8 +1,8 @@
 <?xml version="1.0"?>
 <robot name="robospect" xmlns:xacro="http://www.ros.org/wiki/xacro">
-  <!-- <xacro:include filename="$(find robospect_description)/urdf/bases/robospect_crane.gazebo.xacro" /> -->
+  <xacro:include filename="$(find robospect_description)/urdf/bases/robospect_crane.gazebo.xacro" />
   <xacro:macro name="robospect_crane">
   <!-- FIRST_JOINT -->
-    <joint name="base_first_joint" type="revolute">
+    <joint name="crane_first_joint" type="revolute">
       <axis xyz="0 0 1"/>
       <limit effort="1000.0" lower="-${177.5 * PI / 180}" upper="${177.5 * PI / 180}" velocity="0.5"/>
@@ -11,10 +11,10 @@
       <child link="first_link"/>
     </joint>
-    <transmission name="base_first_joint_trans">
+    <transmission name="crane_first_joint_trans">
       <type>transmission_interface/SimpleTransmission</type>
-      <joint name="base_first_joint">
+      <joint name="crane_first_joint">
         <hardwareInterface>EffortJointInterface</hardwareInterface>
       </joint>
-      <actuator name="base_first_joint_act">
+      <actuator name="crane_first_joint_act">
         <!-- This hardwareInterface element exists for compatibility
              with ROS Hydro. -->
@@ -26,5 +26,5 @@
   <link name="first_link">
     <inertial>
-      <mass value="125.0" />
+      <mass value="12.0" />
       <origin xyz="0 0 0" />
       <inertia  ixx="1.391" ixy="0.004"  ixz="0.0"  iyy="6.853"  iyz="0.0"  izz="6.125" />
@@ -36,5 +36,5 @@
        </geometry>
        <material name="grey">
-          <color rgba="0.8 0.8 0.8 0.95"/>
+          <color rgba="0.8 0.8 0.8 1"/>
        </material>
     </visual>
@@ -46,18 +46,21 @@
     </collision>
   </link>
+  <gazebo reference="first_link">
+    <material>Gazebo/White</material>
+  </gazebo>
   <!-- SECOND_JOINT -->
-    <joint name="base_second_joint" type="prismatic">
+    <joint name="crane_second_joint" type="prismatic">
       <axis xyz="0 0 1"/>
       <limit effort="1000.0" lower="0.0" upper="2.0" velocity="0.5"/>
-      <origin xyz="-0.3 0 1.25" rpy="0 0 0" />  <!-- height is the clearance -->
+      <origin xyz="-0.28 0 1.25" rpy="0 0 0" />  <!-- height is the clearance -->
       <parent link="first_link"/>
       <child link="second_link"/>
     </joint>
-    <transmission name="base_second_joint_trans">
+    <transmission name="crane_second_joint_trans">
       <type>transmission_interface/SimpleTransmission</type>
-      <joint name="base_second_joint">
+      <joint name="crane_second_joint">
         <hardwareInterface>EffortJointInterface</hardwareInterface>
       </joint>
-      <actuator name="base_second_joint_act">
+      <actuator name="crane_second_joint_act">
         <!-- This hardwareInterface element exists for compatibility
              with ROS Hydro. -->
@@ -69,5 +72,5 @@
   <link name="second_link">
     <inertial>
-      <mass value="125.0" />
+      <mass value="2.0" />
       <origin xyz="0 0 0" />
       <inertia  ixx="1.391" ixy="0.004"  ixz="0.0"  iyy="6.853"  iyz="0.0"  izz="6.125" />
@@ -89,17 +92,17 @@
   </link>
     <!-- THIRD_JOINT -->
-      <joint name="base_third_joint" type="revolute">
+      <joint name="crane_third_joint" type="revolute">
         <axis xyz="0 1 0"/>
-        <limit effort="1000.0" lower="-1.2" upper="0.1" velocity="0.5"/>
+        <limit effort="100000.0" lower="-1.2" upper="0.06" velocity="0.2"/>
         <origin xyz="0 0 0" rpy="0 0 0" />  <!-- height is the clearance -->
         <parent link="second_link"/>
         <child link="third_link"/>
       </joint>
-      <transmission name="base_third_joint_trans">
-        <type>transmission_interface/SimpleTransmission</type>
-        <joint name="base_third_joint">
-          <hardwareInterface>EffortJointInterface</hardwareInterface>
-        </joint>
-        <actuator name="base_third_joint_act">
+      <transmission name="crane_third_joint_trans">
+        <type>transmission_interface/SimpleTransmission</type>
+        <joint name="crane_third_joint">
+          <hardwareInterface>EffortJointInterface</hardwareInterface>
+        </joint>
+        <actuator name="crane_third_joint_act">
           <!-- This hardwareInterface element exists for compatibility
                with ROS Hydro. -->
@@ -111,5 +114,5 @@
     <link name="third_link">
       <inertial>
-        <mass value="125.0" />
+        <mass value="2.0" />
         <origin xyz="0 0 0" />
         <inertia  ixx="1.391" ixy="0.004"  ixz="0.0"  iyy="6.853"  iyz="0.0"  izz="6.125" />
@@ -131,17 +134,17 @@
     </link>
     <!-- FOURTH_JOINT -->
-      <joint name="base_fourth_joint" type="prismatic">
+      <joint name="crane_fourth_joint" type="prismatic">
         <axis xyz="1 0 0"/>
         <limit effort="1000.0" lower="0" upper="1.8" velocity="0.5"/>
-        <origin xyz="3.0 0 0" rpy="0 0 0" />  <!-- height is the clearance -->
+        <origin xyz="2.8 0 0.04" rpy="0 0 0" />  <!-- height is the clearance -->
         <parent link="third_link"/>
         <child link="fourth_link"/>
       </joint>
-      <transmission name="base_fourth_joint_trans">
-        <type>transmission_interface/SimpleTransmission</type>
-        <joint name="base_fourth_joint">
-          <hardwareInterface>EffortJointInterface</hardwareInterface>
-        </joint>
-        <actuator name="base_fourth_joint_act">
+      <transmission name="crane_fourth_joint_trans">
+        <type>transmission_interface/SimpleTransmission</type>
+        <joint name="crane_fourth_joint">
+          <hardwareInterface>EffortJointInterface</hardwareInterface>
+        </joint>
+        <actuator name="crane_fourth_joint_act">
           <!-- This hardwareInterface element exists for compatibility
                with ROS Hydro. -->
@@ -153,5 +156,5 @@
     <link name="fourth_link">
       <inertial>
-        <mass value="125.0" />
+        <mass value="2.0" />
         <origin xyz="0 0 0" />
         <inertia  ixx="1.391" ixy="0.004"  ixz="0.0"  iyy="6.853"  iyz="0.0"  izz="6.125" />
@@ -173,17 +176,17 @@
     </link>
     <!-- FIFTH_JOINT -->
-      <joint name="base_fifth_joint" type="revolute">
+      <joint name="crane_fifth_joint" type="revolute">
         <axis xyz="0 1 0"/>
-        <limit effort="1000.0" lower="-0.5" upper="0.6" velocity="0.5"/>
+        <limit effort="1000.0" lower="-0.7" upper="0.6" velocity="0.5"/>
         <origin xyz="0 0 0" rpy="0 0 0" />  <!-- height is the clearance -->
         <parent link="fourth_link"/>
         <child link="fifth_link"/>
       </joint>
-      <transmission name="base_fifth_joint_trans">
-        <type>transmission_interface/SimpleTransmission</type>
-        <joint name="base_fifth_joint">
-          <hardwareInterface>EffortJointInterface</hardwareInterface>
-        </joint>
-        <actuator name="base_fifth_joint_act">
+      <transmission name="crane_fifth_joint_trans">
+        <type>transmission_interface/SimpleTransmission</type>
+        <joint name="crane_fifth_joint">
+          <hardwareInterface>EffortJointInterface</hardwareInterface>
+        </joint>
+        <actuator name="crane_fifth_joint_act">
           <!-- This hardwareInterface element exists for compatibility
                with ROS Hydro. -->
@@ -195,5 +198,5 @@
     <link name="fifth_link">
       <inertial>
-        <mass value="125.0" />
+        <mass value="2.0" />
         <origin xyz="0 0 0" />
         <inertia  ixx="1.391" ixy="0.004"  ixz="0.0"  iyy="6.853"  iyz="0.0"  izz="6.125" />
@@ -215,17 +218,17 @@
     </link>
     <!-- SIXTH_JOINT -->
-      <joint name="base_sixth_joint" type="revolute">
+      <joint name="crane_sixth_joint" type="revolute">
         <axis xyz="0 1 0"/>
-        <limit effort="1000.0" lower="0" upper="1.5" velocity="0.5"/>
+        <limit effort="1000.0" lower="-0.5" upper="1.5" velocity="0.5"/>
         <origin xyz="0.25415 0 0" rpy="0 0 0" />  <!-- height is the clearance -->
         <parent link="fifth_link"/>
         <child link="sixth_link"/>
       </joint>
-      <transmission name="base_sixth_joint_trans">
-        <type>transmission_interface/SimpleTransmission</type>
-        <joint name="base_sixth_joint">
-          <hardwareInterface>EffortJointInterface</hardwareInterface>
-        </joint>
-        <actuator name="base_sixth_joint_act">
+      <transmission name="crane_sixth_joint_trans">
+        <type>transmission_interface/SimpleTransmission</type>
+        <joint name="crane_sixth_joint">
+          <hardwareInterface>EffortJointInterface</hardwareInterface>
+        </joint>
+        <actuator name="crane_sixth_joint_act">
           <!-- This hardwareInterface element exists for compatibility
                with ROS Hydro. -->
@@ -237,5 +240,5 @@
     <link name="sixth_link">
       <inertial>
-        <mass value="125.0" />
+        <mass value="1.0" />
         <origin xyz="0 0 0" />
         <inertia  ixx="1.391" ixy="0.004"  ixz="0.0"  iyy="6.853"  iyz="0.0"  izz="6.125" />
@@ -257,5 +260,5 @@
     </link>
     <!-- SIXTH_AUX_JOINT -->
-      <joint name="base_sixth_aux_joint" type="revolute">
+      <joint name="crane_sixth_aux_joint" type="revolute">
         <axis xyz="0 1 0"/>
         <limit effort="1000.0" lower="0" upper="1.3" velocity="0.5"/>
@@ -263,12 +266,12 @@
         <parent link="fifth_link"/>
         <child link="sixth_aux_link"/>
-        <mimic joint="base_sixth_joint"/>
-      </joint>
-      <transmission name="base_sixth_aux_joint_trans">
-        <type>transmission_interface/SimpleTransmission</type>
-        <joint name="base_sixth_joint">
-          <hardwareInterface>EffortJointInterface</hardwareInterface>
-        </joint>
-        <actuator name="base_sixth_aux_joint_act">
+        <mimic joint="crane_sixth_joint"/>
+      </joint>
+      <transmission name="crane_sixth_aux_joint_trans">
+        <type>transmission_interface/SimpleTransmission</type>
+        <joint name="crane_sixth_joint">
+          <hardwareInterface>EffortJointInterface</hardwareInterface>
+        </joint>
+        <actuator name="crane_sixth_aux_joint_act">
           <!-- This hardwareInterface element exists for compatibility
                with ROS Hydro. -->
@@ -280,5 +283,5 @@
     <link name="sixth_aux_link">
       <inertial>
-        <mass value="125.0" />
+        <mass value="1.0" />
         <origin xyz="0 0 0" />
         <inertia  ixx="1.391" ixy="0.004"  ixz="0.0"  iyy="6.853"  iyz="0.0"  izz="6.125" />
@@ -300,5 +303,5 @@
     </link>
     <!-- SEVENTH_JOINT -->
-      <joint name="base_seventh_joint" type="revolute">
+      <joint name="crane_seventh_joint" type="revolute">
         <axis xyz="0 0 1"/>
         <limit effort="1000.0" lower="-${90 * PI / 180}" upper="${90 * PI / 180}" velocity="0.5"/>
@@ -306,12 +309,12 @@
         <parent link="sixth_link"/>
         <child link="seventh_link"/>
-        <mimic joint="base_sixth_joint" offset="-0.485"/>
-      </joint>
-      <transmission name="base_seventh_joint_trans">
-        <type>transmission_interface/SimpleTransmission</type>
-        <joint name="base_seventh_joint">
-          <hardwareInterface>EffortJointInterface</hardwareInterface>
-        </joint>
-        <actuator name="base_seventh_joint_act">
+        <mimic joint="crane_sixth_joint" offset="-0.485"/>
+      </joint>
+      <transmission name="crane_seventh_joint_trans">
+        <type>transmission_interface/SimpleTransmission</type>
+        <joint name="crane_seventh_joint">
+          <hardwareInterface>EffortJointInterface</hardwareInterface>
+        </joint>
+        <actuator name="crane_seventh_joint_act">
           <!-- This hardwareInterface element exists for compatibility
                with ROS Hydro. -->
@@ -323,5 +326,5 @@
     <link name="seventh_link">
       <inertial>
-        <mass value="125.0" />
+        <mass value="1.0" />
         <origin xyz="0 0 0" />
         <inertia  ixx="1.391" ixy="0.004"  ixz="0.0"  iyy="6.853"  iyz="0.0"  izz="6.125" />
@@ -343,5 +346,5 @@
     </link>
     <!-- TIP_JOINT -->
-      <joint name="base_tip_joint" type="revolute">
+      <joint name="crane_tip_joint" type="revolute">
         <axis xyz="0 0 1"/>
         <limit effort="1000.0" lower="-${90 * PI / 180}" upper="${90 * PI / 180}" velocity="0.5"/>
@@ -350,10 +353,10 @@
         <child link="tip_link"/>
       </joint>
-      <transmission name="base_tip_joint_trans">
-        <type>transmission_interface/SimpleTransmission</type>
-        <joint name="base_tip_joint">
-          <hardwareInterface>EffortJointInterface</hardwareInterface>
-        </joint>
-        <actuator name="base_tip_joint_act">
+      <transmission name="crane_tip_joint_trans">
+        <type>transmission_interface/SimpleTransmission</type>
+        <joint name="crane_tip_joint">
+          <hardwareInterface>EffortJointInterface</hardwareInterface>
+        </joint>
+        <actuator name="crane_tip_joint_act">
           <!-- This hardwareInterface element exists for compatibility
                with ROS Hydro. -->
@@ -365,5 +368,5 @@
     <link name="tip_link">
       <inertial>
-        <mass value="125.0" />
+        <mass value="1.0" />
         <origin xyz="0 0 0" />
         <inertia  ixx="1.391" ixy="0.004"  ixz="0.0"  iyy="6.853"  iyz="0.0"  izz="6.125" />

File: robospect_description/urdf/wheels/suspension_wheel.urdf.xacro (robot description, xacro)
@@ -9,5 +9,5 @@
   <xacro:property name="tire_dia" value="0.56"/>
   <xacro:property name="tire_width" value="0.2"/>
-  <xacro:property name="hex_hub_depth" value="0.120"/> <!-- or +0.072 -->
+  <xacro:property name="hex_hub_depth" value="0.12"/> <!-- or +0.072 -->
   <xacro:property name="wheel_mass" value="15.0"/>   <!-- check -->
   <!-- hex_hub_dist is the distance between left and right hex hubs when
@@ -16,8 +16,9 @@
        vertical wheel travel. -->
   <xacro:property name="wheelbase" value="1.6"/>
+  <xacro:property name="wheelbase_rear" value="1.0"/>
   <xacro:property name="hex_hub_dist" value="0.900"/>  <!-- 1.127 0.742 check -->
-  <xacro:property name="axle_length" value="0.120"/>
-  <xacro:property name="wheel_travel" value="0.1"/>
-  <xacro:property name="shock_z_offset" value="0.05"/>
+  <xacro:property name="axle_length" value="0.01"/>
+  <xacro:property name="wheel_travel" value="0.001"/>
+  <xacro:property name="shock_z_offset" value="0.001"/>
   <!-- Degree-to-radian conversions -->
   <xacro:property name="degrees_45" value="0.785398163"/>
@@ -25,6 +26,6 @@
   <xacro:property name="degrees_180" value="3.14159265"/>
   <!-- shock_eff_limit is 2 * ((shock_stroke / 2) * shock_spring_constant) N. -->
-  <xacro:property name="shock_eff_limit" value="100"/>
-  <xacro:property name="shock_vel_limit" value="1000"/>
+  <xacro:property name="shock_eff_limit" value="10000"/>
+  <xacro:property name="shock_vel_limit" value="1"/>
   <!-- axle eff limit = 2 * stall_torque
        as a function of the max gradient (15%) with overall max payload (600Kg) * wheel_radius
@@ -32,5 +33,5 @@
        axle_eff_limit = 204.95 / 2 N m = ~102.5 -->
   <!-- xacro:property name="axle_eff_limit" value="102.5"/ -->
-  <xacro:property name="axle_eff_limit" value="204.95"/>
+  <xacro:property name="axle_eff_limit" value="200.0"/>
   <!-- max_speed = 33 Km/h = 9.17 m/s
        axle_vel_limit = (2 * pi) * (max_speed / (pi * tire_dia)) =  39.02 rad/s -->
@@ -130,5 +131,5 @@
     </transmission>
     <gazebo reference="${lr_prefix}_${fr_prefix}_axle_carrier">
-      <material>Gazebo/White</material>
+      <material>Gazebo/Grey</material>
     </gazebo>
     <link name="${lr_prefix}_${fr_prefix}_wheel">
@@ -138,5 +139,6 @@
                      ${lr_reflect * (axle_length - (tire_width / 2 - hex_hub_depth))}"/>
         <geometry>
-          <cylinder radius="${tire_dia / 2}" length="${tire_width}"/>
+          <!--<cylinder radius="${tire_dia / 2}" length="${tire_width}"/> -->
+          <mesh filename="package://robospect_description/meshes/wheels/robospect_wheel_l.STL" scale="1 1 1"/>
         </geometry>
         <material name="tire_mat"/>
@@ -147,5 +149,6 @@
                      ${lr_reflect * (axle_length - (tire_width / 2 - hex_hub_depth))}"/>
         <geometry>
-          <cylinder radius="${tire_dia / 2}" length="${tire_width}"/>
+          <!--<cylinder radius="${tire_dia / 2}" length="${tire_width}"/> -->
+          <mesh filename="package://robospect_description/meshes/wheels/robospect_wheel_l.STL" scale="1 1 1"/>
         </geometry>
       </collision>
@@ -155,8 +158,7 @@
     </link>
     <gazebo reference="${lr_prefix}_${fr_prefix}_wheel">
-      <material>Gazebo/White</material>
+      <material>Gazebo/Grey</material>
     </gazebo>
   </xacro:macro>
-  <!-- xacro:macro name="rubber_wheel" params="name parent *origin reflect hq" -->
   <!-- Front wheel -->
   <xacro:macro name="front_wheel"
@@ -200,5 +202,5 @@
     </transmission>
     <gazebo reference="${lr_prefix}_steering_link">
-      <material>Gazebo/White</material>
+      <material>Gazebo/Grey</material>
     </gazebo>
     <xacro:wheel lr_prefix="${lr_prefix}" fr_prefix="${fr_prefix}"

Commit message: New test settings

File: robospect_description/urdf/bases/robospect_base.urdf.xacro (robot description, xacro)
@@ -32,5 +32,5 @@
   <link name="base_link">
     <inertial>
-      <mass value="200.0" />
+      <mass value="500.0" />
       <origin xyz="0 0 0" />
       <inertia  ixx="1.391" ixy="0.004"  ixz="0.0"  iyy="6.853"  iyz="0.0"  izz="6.125" />

File: robospect_description/urdf/wheels/standard_wheel.urdf.xacro (robot description, xacro)
@@ -1,6 +1,6 @@
 <?xml version="1.0"?>
 <robot name="wheel" xmlns:xacro="http://www.ros.org/wiki/xacro">
-  <xacro:property name="wheel_offset_x" value="0.750" />    <!-- x,y,z in base_footprint CS -->
-  <xacro:property name="wheel_offset_y" value="0.553" />
+  <xacro:property name="wheel_offset_x" value="0.800" />    <!-- x,y,z in base_footprint CS -->
+  <xacro:property name="wheel_offset_y" value="0.56" />
   <xacro:property name="wheel_offset_z" value="0.0" />
   <xacro:property name="wheel_joint_damping" value="1.0" />
@@ -81,6 +81,6 @@
 		<inertial>
 			<origin xyz="0 0 0" />
-			<mass value="0.001"/>
-			<inertia ixx="0.001" ixy="0" ixz="0" iyy="0.001" iyz="0" izz="0.001"/>
+			<mass value="5.0"/>
+			<inertia  ixx="0.01" ixy="0.0"  ixz="0.0"  iyy="0.01"  iyz="0.0"  izz="0.01" />
 		</inertial>
     </link>
