Commit message: description: Replacing .stl by .dae

File: robospect_description/urdf/bases/robospect_base.urdf.xacro (robot description, xacro)
@@ -39,5 +39,5 @@
        <origin xyz="0 0 0" rpy="0 0 0" />
        <geometry>
-	       <mesh filename="package://robospect_description/meshes/bases/robospect_base_chassis.STL"/>
+	       <mesh filename="package://robospect_description/meshes/bases/robospect_base_chassis.dae"/>
        </geometry>
        <material name="blue">
@@ -48,5 +48,5 @@
        <origin xyz="0 0 0" rpy="0 0 0" />
        <geometry>
-         <mesh filename="package://robospect_description/meshes/bases/robospect_base_chassis.STL"/>
+         <mesh filename="package://robospect_description/meshes/bases/robospect_base_chassis.dae"/>
        </geometry>
     </collision>

File: robospect_description/urdf/bases/robospect_crane.urdf.xacro (robot description, xacro)
@@ -47,5 +47,5 @@
        <origin xyz="0 0 0" rpy="0 0 0" />
        <geometry>
-	        <mesh filename="package://robospect_description/meshes/bases/robospect_first.STL" scale="1 1 1"/>
+	        <mesh filename="package://robospect_description/meshes/bases/robospect_first.dae" scale="1 1 1"/>
        </geometry>
        <material name="grey">
@@ -56,5 +56,5 @@
        <origin xyz="0 0 0" rpy="0 0 0 " />
        <geometry>
-         <mesh filename="package://robospect_description/meshes/bases/robospect_first.STL" scale="1 1 1"/>
+         <mesh filename="package://robospect_description/meshes/bases/robospect_first.dae" scale="1 1 1"/>
        </geometry>
     </collision>
@@ -93,5 +93,5 @@
        <origin xyz="0 0 0" rpy="0 0 0" />
        <geometry>
-	        <mesh filename="package://robospect_description/meshes/bases/robospect_second.STL" scale="1 1 1"/>
+	        <mesh filename="package://robospect_description/meshes/bases/robospect_second.dae" scale="1 1 1"/>
        </geometry>
        <material name="blue">
@@ -101,5 +101,5 @@
        <origin xyz="0 0 0" rpy="0 0 0 " />
        <geometry>
-         <mesh filename="package://robospect_description/meshes/bases/robospect_second.STL" scale="1 1 1"/>
+         <mesh filename="package://robospect_description/meshes/bases/robospect_second.dae" scale="1 1 1"/>
        </geometry>
     </collision>
@@ -133,13 +133,13 @@
          <origin xyz="0 0 0" rpy="0 0 0" />
          <geometry>
-  	        <mesh filename="package://robospect_description/meshes/bases/robospect_third.STL" scale="1 1 1"/>
-         </geometry>
-         <material name="blue">
-         </material>
-      </visual>
-      <collision>
-         <origin xyz="0 0 0" rpy="0 0 0 " />
-         <geometry>
-           <mesh filename="package://robospect_description/meshes/bases/robospect_third.STL" scale="1 1 1"/>
+  	        <mesh filename="package://robospect_description/meshes/bases/robospect_third.dae" scale="1 1 1"/>
+         </geometry>
+         <material name="blue">
+         </material>
+      </visual>
+      <collision>
+         <origin xyz="0 0 0" rpy="0 0 0 " />
+         <geometry>
+           <mesh filename="package://robospect_description/meshes/bases/robospect_third.dae" scale="1 1 1"/>
          </geometry>
       </collision>
@@ -174,13 +174,13 @@
          <origin xyz="0 0 0" rpy="0 0 0" />
          <geometry>
-            <mesh filename="package://robospect_description/meshes/bases/robospect_fourth.STL" scale="1 1 1"/>
-         </geometry>
-         <material name="blue">
-         </material>
-      </visual>
-      <collision>
-         <origin xyz="0 0 0" rpy="0 0 0 " />
-         <geometry>
-           <mesh filename="package://robospect_description/meshes/bases/robospect_fourth.STL" scale="1 1 1"/>
+            <mesh filename="package://robospect_description/meshes/bases/robospect_fourth.dae" scale="1 1 1"/>
+         </geometry>
+         <material name="blue">
+         </material>
+      </visual>
+      <collision>
+         <origin xyz="0 0 0" rpy="0 0 0 " />
+         <geometry>
+           <mesh filename="package://robospect_description/meshes/bases/robospect_fourth.dae" scale="1 1 1"/>
          </geometry>
       </collision>
@@ -214,13 +214,13 @@
          <origin xyz="0 0 0" rpy="0 0 0" />
          <geometry>
-            <mesh filename="package://robospect_description/meshes/bases/robospect_fifth.STL" scale="1 1 1"/>
-         </geometry>
-         <material name="blue">
-         </material>
-      </visual>
-      <collision>
-         <origin xyz="0 0 0" rpy="0 0 0 " />
-         <geometry>
-           <mesh filename="package://robospect_description/meshes/bases/robospect_fifth.STL" scale="1 1 1"/>
+            <mesh filename="package://robospect_description/meshes/bases/robospect_fifth.dae" scale="1 1 1"/>
+         </geometry>
+         <material name="blue">
+         </material>
+      </visual>
+      <collision>
+         <origin xyz="0 0 0" rpy="0 0 0 " />
+         <geometry>
+           <mesh filename="package://robospect_description/meshes/bases/robospect_fifth.dae" scale="1 1 1"/>
          </geometry>
       </collision>
@@ -280,13 +280,13 @@
          <origin xyz="0 0 0" rpy="0 0 0" />
          <geometry>
-            <mesh filename="package://robospect_description/meshes/bases/robospect_sixth.STL" scale="1 1 1"/>
-         </geometry>
-         <material name="blue">
-         </material>
-      </visual>
-      <collision>
-         <origin xyz="0 0 0" rpy="0 0 0 " />
-         <geometry>
-           <mesh filename="package://robospect_description/meshes/bases/robospect_sixth.STL" scale="1 1 1"/>
+            <mesh filename="package://robospect_description/meshes/bases/robospect_sixth.dae" scale="1 1 1"/>
+         </geometry>
+         <material name="blue">
+         </material>
+      </visual>
+      <collision>
+         <origin xyz="0 0 0" rpy="0 0 0 " />
+         <geometry>
+           <mesh filename="package://robospect_description/meshes/bases/robospect_sixth.dae" scale="1 1 1"/>
          </geometry>
       </collision>
@@ -320,13 +320,13 @@
          <origin xyz="0 0 0" rpy="0 0 0" />
          <geometry>
-            <mesh filename="package://robospect_description/meshes/bases/robospect_sixth.STL" scale="1 1 1"/>
-         </geometry>
-         <material name="blue">
-         </material>
-      </visual>
-      <collision>
-         <origin xyz="0 0 0" rpy="0 0 0 " />
-         <geometry>
-           <mesh filename="package://robospect_description/meshes/bases/robospect_sixth.STL" scale="1 1 1"/>
+            <mesh filename="package://robospect_description/meshes/bases/robospect_sixth.dae" scale="1 1 1"/>
+         </geometry>
+         <material name="blue">
+         </material>
+      </visual>
+      <collision>
+         <origin xyz="0 0 0" rpy="0 0 0 " />
+         <geometry>
+           <mesh filename="package://robospect_description/meshes/bases/robospect_sixth.dae" scale="1 1 1"/>
          </geometry>
       </collision>
@@ -360,13 +360,13 @@
          <origin xyz="0 0 0" rpy="0 0 0" />
          <geometry>
-            <mesh filename="package://robospect_description/meshes/bases/robospect_sixth.STL" scale="1 1 1"/>
-         </geometry>
-         <material name="blue">
-         </material>
-      </visual>
-      <collision>
-         <origin xyz="0 0 0" rpy="0 0 0 " />
-         <geometry>
-           <mesh filename="package://robospect_description/meshes/bases/robospect_sixth.STL" scale="1 1 1"/>
+            <mesh filename="package://robospect_description/meshes/bases/robospect_sixth.dae" scale="1 1 1"/>
+         </geometry>
+         <material name="blue">
+         </material>
+      </visual>
+      <collision>
+         <origin xyz="0 0 0" rpy="0 0 0 " />
+         <geometry>
+           <mesh filename="package://robospect_description/meshes/bases/robospect_sixth.dae" scale="1 1 1"/>
          </geometry>
       </collision>
@@ -400,13 +400,13 @@
          <origin xyz="0 0 0" rpy="0 0 0" />
          <geometry>
-            <mesh filename="package://robospect_description/meshes/bases/robospect_sixth.STL" scale="1 1 1"/>
-         </geometry>
-         <material name="blue">
-         </material>
-      </visual>
-      <collision>
-         <origin xyz="0 0 0" rpy="0 0 0 " />
-         <geometry>
-           <mesh filename="package://robospect_description/meshes/bases/robospect_sixth.STL" scale="1 1 1"/>
+            <mesh filename="package://robospect_description/meshes/bases/robospect_sixth.dae" scale="1 1 1"/>
+         </geometry>
+         <material name="blue">
+         </material>
+      </visual>
+      <collision>
+         <origin xyz="0 0 0" rpy="0 0 0 " />
+         <geometry>
+           <mesh filename="package://robospect_description/meshes/bases/robospect_sixth.dae" scale="1 1 1"/>
          </geometry>
       </collision>
@@ -443,13 +443,13 @@
          <origin xyz="0 0 0" rpy="0 0 0" />
          <geometry>
-            <mesh filename="package://robospect_description/meshes/bases/robospect_seventh.STL" scale="1 1 1"/>
-         </geometry>
-         <material name="blue">
-         </material>
-      </visual>
-      <collision>
-         <origin xyz="0 0 0" rpy="0 0 0 " />
-         <geometry>
-           <mesh filename="package://robospect_description/meshes/bases/robospect_seventh.STL" scale="1 1 1"/>
+            <mesh filename="package://robospect_description/meshes/bases/robospect_seventh.dae" scale="1 1 1"/>
+         </geometry>
+         <material name="blue">
+         </material>
+      </visual>
+      <collision>
+         <origin xyz="0 0 0" rpy="0 0 0 " />
+         <geometry>
+           <mesh filename="package://robospect_description/meshes/bases/robospect_seventh.dae" scale="1 1 1"/>
          </geometry>
       </collision>
@@ -483,5 +483,5 @@
          <origin xyz="0 0 0" rpy="0 0 0" />
          <geometry>
-            <mesh filename="package://robospect_description/meshes/bases/robospect_head.STL" scale="1 1 1"/>
+            <mesh filename="package://robospect_description/meshes/bases/robospect_head.dae" scale="1 1 1"/>
          </geometry>
          <material name="black">
@@ -491,5 +491,5 @@
          <origin xyz="0 0 0" rpy="0 0 0 " />
          <geometry>
-           <mesh filename="package://robospect_description/meshes/bases/robospect_head.STL" scale="1 1 1"/>
+           <mesh filename="package://robospect_description/meshes/bases/robospect_head.dae" scale="1 1 1"/>
          </geometry>
       </collision>

File: robospect_description/urdf/wheels/standard_wheel.urdf.xacro (robot description, xacro)
@@ -43,5 +43,5 @@
         <origin xyz="${x_link_offset} ${y_link_offset} ${z_link_offset}"/>
         <geometry>
-          <mesh filename="package://robospect_description/meshes/wheels/robospect_wheel_l.STL" scale="1 1 1"/>
+          <mesh filename="package://robospect_description/meshes/wheels/robospect_wheel_l.dae" scale="1 1 1"/>
           <!--mesh filename="package://robospect_description/meshes/wheels/rbcar_wheel1.stl" scale="1 1 1"/-->
         </geometry>
@@ -51,5 +51,5 @@
         <origin xyz="${x_link_offset} ${y_link_offset} ${z_link_offset}"/>
         <geometry>
-          <mesh filename="package://robospect_description/meshes/wheels/robospect_wheel_l.STL" scale="1 1 1"/>
+          <mesh filename="package://robospect_description/meshes/wheels/robospect_wheel_l.dae" scale="1 1 1"/>
         </geometry>
       </collision>
