Commit message: Double bar and TIp included.

File: robospect_description/urdf/bases/robospect_crane.urdf.xacro (robot description, xacro)
@@ -6,5 +6,5 @@
     <joint name="base_first_joint" type="revolute">
       <axis xyz="0 0 1"/>
-      <limit effort="1000.0" lower="-${90 * PI / 180}" upper="${90 * PI / 180}" velocity="0.5"/>
+      <limit effort="1000.0" lower="-${177.5 * PI / 180}" upper="${177.5 * PI / 180}" velocity="0.5"/>
       <origin xyz="-0.046851 0 0.3" rpy="0 0 0" />  <!-- height is the clearance -->
       <parent link="base_link"/>
@@ -88,4 +88,300 @@
     </collision>
   </link>
+    <!-- THIRD_JOINT -->
+      <joint name="base_third_joint" type="revolute">
+        <axis xyz="0 1 0"/>
+        <limit effort="1000.0" lower="-1.2" upper="0.1" velocity="0.5"/>
+        <origin xyz="0 0 0" rpy="0 0 0" />  <!-- height is the clearance -->
+        <parent link="second_link"/>
+        <child link="third_link"/>
+      </joint>
+      <transmission name="base_third_joint_trans">
+        <type>transmission_interface/SimpleTransmission</type>
+        <joint name="base_third_joint">
+          <hardwareInterface>EffortJointInterface</hardwareInterface>
+        </joint>
+        <actuator name="base_third_joint_act">
+          <!-- This hardwareInterface element exists for compatibility
+               with ROS Hydro. -->
+          <hardwareInterface>EffortJointInterface</hardwareInterface>
+          <mechanicalReduction>1</mechanicalReduction>
+        </actuator>
+      </transmission>
+    <!-- THIRD_LINK -->
+    <link name="third_link">
+      <inertial>
+        <mass value="125.0" />
+        <origin xyz="0 0 0" />
+        <inertia  ixx="1.391" ixy="0.004"  ixz="0.0"  iyy="6.853"  iyz="0.0"  izz="6.125" />
+      </inertial>
+      <visual>
+         <origin xyz="0 0 0" rpy="0 0 0" />
+         <geometry>
+  	        <mesh filename="package://robospect_description/meshes/bases/robospect_third.STL" scale="1 1 1"/>
+         </geometry>
+         <material name="blue">
+         </material>
+      </visual>
+      <collision>
+         <origin xyz="0 0 0" rpy="0 0 0 " />
+         <geometry>
+           <mesh filename="package://robospect_description/meshes/bases/robospect_third.STL" scale="1 1 1"/>
+         </geometry>
+      </collision>
+    </link>
+    <!-- FOURTH_JOINT -->
+      <joint name="base_fourth_joint" type="prismatic">
+        <axis xyz="1 0 0"/>
+        <limit effort="1000.0" lower="0" upper="1.8" velocity="0.5"/>
+        <origin xyz="3.0 0 0" rpy="0 0 0" />  <!-- height is the clearance -->
+        <parent link="third_link"/>
+        <child link="fourth_link"/>
+      </joint>
+      <transmission name="base_fourth_joint_trans">
+        <type>transmission_interface/SimpleTransmission</type>
+        <joint name="base_fourth_joint">
+          <hardwareInterface>EffortJointInterface</hardwareInterface>
+        </joint>
+        <actuator name="base_fourth_joint_act">
+          <!-- This hardwareInterface element exists for compatibility
+               with ROS Hydro. -->
+          <hardwareInterface>EffortJointInterface</hardwareInterface>
+          <mechanicalReduction>1</mechanicalReduction>
+        </actuator>
+      </transmission>
+    <!-- FOURTH_LINK -->
+    <link name="fourth_link">
+      <inertial>
+        <mass value="125.0" />
+        <origin xyz="0 0 0" />
+        <inertia  ixx="1.391" ixy="0.004"  ixz="0.0"  iyy="6.853"  iyz="0.0"  izz="6.125" />
+      </inertial>
+      <visual>
+         <origin xyz="0 0 0" rpy="0 0 0" />
+         <geometry>
+            <mesh filename="package://robospect_description/meshes/bases/robospect_fourth.STL" scale="1 1 1"/>
+         </geometry>
+         <material name="blue">
+         </material>
+      </visual>
+      <collision>
+         <origin xyz="0 0 0" rpy="0 0 0 " />
+         <geometry>
+           <mesh filename="package://robospect_description/meshes/bases/robospect_fourth.STL" scale="1 1 1"/>
+         </geometry>
+      </collision>
+    </link>
+    <!-- FIFTH_JOINT -->
+      <joint name="base_fifth_joint" type="revolute">
+        <axis xyz="0 1 0"/>
+        <limit effort="1000.0" lower="-0.5" upper="0.6" velocity="0.5"/>
+        <origin xyz="0 0 0" rpy="0 0 0" />  <!-- height is the clearance -->
+        <parent link="fourth_link"/>
+        <child link="fifth_link"/>
+      </joint>
+      <transmission name="base_fifth_joint_trans">
+        <type>transmission_interface/SimpleTransmission</type>
+        <joint name="base_fifth_joint">
+          <hardwareInterface>EffortJointInterface</hardwareInterface>
+        </joint>
+        <actuator name="base_fifth_joint_act">
+          <!-- This hardwareInterface element exists for compatibility
+               with ROS Hydro. -->
+          <hardwareInterface>EffortJointInterface</hardwareInterface>
+          <mechanicalReduction>1</mechanicalReduction>
+        </actuator>
+      </transmission>
+    <!-- FIFTH_LINK -->
+    <link name="fifth_link">
+      <inertial>
+        <mass value="125.0" />
+        <origin xyz="0 0 0" />
+        <inertia  ixx="1.391" ixy="0.004"  ixz="0.0"  iyy="6.853"  iyz="0.0"  izz="6.125" />
+      </inertial>
+      <visual>
+         <origin xyz="0 0 0" rpy="0 0 0" />
+         <geometry>
+            <mesh filename="package://robospect_description/meshes/bases/robospect_fifth.STL" scale="1 1 1"/>
+         </geometry>
+         <material name="blue">
+         </material>
+      </visual>
+      <collision>
+         <origin xyz="0 0 0" rpy="0 0 0 " />
+         <geometry>
+           <mesh filename="package://robospect_description/meshes/bases/robospect_fifth.STL" scale="1 1 1"/>
+         </geometry>
+      </collision>
+    </link>
+    <!-- SIXTH_JOINT -->
+      <joint name="base_sixth_joint" type="revolute">
+        <axis xyz="0 1 0"/>
+        <limit effort="1000.0" lower="0" upper="1.5" velocity="0.5"/>
+        <origin xyz="0.25415 0 0" rpy="0 0 0" />  <!-- height is the clearance -->
+        <parent link="fifth_link"/>
+        <child link="sixth_link"/>
+      </joint>
+      <transmission name="base_sixth_joint_trans">
+        <type>transmission_interface/SimpleTransmission</type>
+        <joint name="base_sixth_joint">
+          <hardwareInterface>EffortJointInterface</hardwareInterface>
+        </joint>
+        <actuator name="base_sixth_joint_act">
+          <!-- This hardwareInterface element exists for compatibility
+               with ROS Hydro. -->
+          <hardwareInterface>EffortJointInterface</hardwareInterface>
+          <mechanicalReduction>1</mechanicalReduction>
+        </actuator>
+      </transmission>
+    <!-- SIXTH_LINK -->
+    <link name="sixth_link">
+      <inertial>
+        <mass value="125.0" />
+        <origin xyz="0 0 0" />
+        <inertia  ixx="1.391" ixy="0.004"  ixz="0.0"  iyy="6.853"  iyz="0.0"  izz="6.125" />
+      </inertial>
+      <visual>
+         <origin xyz="0 0 0" rpy="0 0 0" />
+         <geometry>
+            <mesh filename="package://robospect_description/meshes/bases/robospect_sixth.STL" scale="1 1 1"/>
+         </geometry>
+         <material name="blue">
+         </material>
+      </visual>
+      <collision>
+         <origin xyz="0 0 0" rpy="0 0 0 " />
+         <geometry>
+           <mesh filename="package://robospect_description/meshes/bases/robospect_sixth.STL" scale="1 1 1"/>
+         </geometry>
+      </collision>
+    </link>
+    <!-- SIXTH_AUX_JOINT -->
+      <joint name="base_sixth_aux_joint" type="revolute">
+        <axis xyz="0 1 0"/>
+        <limit effort="1000.0" lower="0" upper="1.3" velocity="0.5"/>
+        <origin xyz="0.1177 0 -0.26422" rpy="0 0 0" />  <!-- height is the clearance -->
+        <parent link="fifth_link"/>
+        <child link="sixth_aux_link"/>
+        <mimic joint="base_sixth_joint"/>
+      </joint>
+      <transmission name="base_sixth_aux_joint_trans">
+        <type>transmission_interface/SimpleTransmission</type>
+        <joint name="base_sixth_joint">
+          <hardwareInterface>EffortJointInterface</hardwareInterface>
+        </joint>
+        <actuator name="base_sixth_aux_joint_act">
+          <!-- This hardwareInterface element exists for compatibility
+               with ROS Hydro. -->
+          <hardwareInterface>EffortJointInterface</hardwareInterface>
+          <mechanicalReduction>1</mechanicalReduction>
+        </actuator>
+      </transmission>
+    <!-- SIXTH_AUX_LINK -->
+    <link name="sixth_aux_link">
+      <inertial>
+        <mass value="125.0" />
+        <origin xyz="0 0 0" />
+        <inertia  ixx="1.391" ixy="0.004"  ixz="0.0"  iyy="6.853"  iyz="0.0"  izz="6.125" />
+      </inertial>
+      <visual>
+         <origin xyz="0 0 0" rpy="0 0 0" />
+         <geometry>
+            <mesh filename="package://robospect_description/meshes/bases/robospect_sixth.STL" scale="1 1 1"/>
+         </geometry>
+         <material name="blue">
+         </material>
+      </visual>
+      <collision>
+         <origin xyz="0 0 0" rpy="0 0 0 " />
+         <geometry>
+           <mesh filename="package://robospect_description/meshes/bases/robospect_sixth.STL" scale="1 1 1"/>
+         </geometry>
+      </collision>
+    </link>
+    <!-- SEVENTH_JOINT -->
+      <joint name="base_seventh_joint" type="revolute">
+        <axis xyz="0 0 1"/>
+        <limit effort="1000.0" lower="-${90 * PI / 180}" upper="${90 * PI / 180}" velocity="0.5"/>
+        <origin xyz="2.0 0 0" rpy="${90 * PI / 180} 0 0" />  <!-- height is the clearance -->
+        <parent link="sixth_link"/>
+        <child link="seventh_link"/>
+        <mimic joint="base_sixth_joint" offset="-0.485"/>
+      </joint>
+      <transmission name="base_seventh_joint_trans">
+        <type>transmission_interface/SimpleTransmission</type>
+        <joint name="base_seventh_joint">
+          <hardwareInterface>EffortJointInterface</hardwareInterface>
+        </joint>
+        <actuator name="base_seventh_joint_act">
+          <!-- This hardwareInterface element exists for compatibility
+               with ROS Hydro. -->
+          <hardwareInterface>EffortJointInterface</hardwareInterface>
+          <mechanicalReduction>1</mechanicalReduction>
+        </actuator>
+      </transmission>
+    <!-- SEVENTH_LINK -->
+    <link name="seventh_link">
+      <inertial>
+        <mass value="125.0" />
+        <origin xyz="0 0 0" />
+        <inertia  ixx="1.391" ixy="0.004"  ixz="0.0"  iyy="6.853"  iyz="0.0"  izz="6.125" />
+      </inertial>
+      <visual>
+         <origin xyz="0 0 0" rpy="0 0 0" />
+         <geometry>
+            <mesh filename="package://robospect_description/meshes/bases/robospect_seventh.STL" scale="1 1 1"/>
+         </geometry>
+         <material name="blue">
+         </material>
+      </visual>
+      <collision>
+         <origin xyz="0 0 0" rpy="0 0 0 " />
+         <geometry>
+           <mesh filename="package://robospect_description/meshes/bases/robospect_seventh.STL" scale="1 1 1"/>
+         </geometry>
+      </collision>
+    </link>
+    <!-- TIP_JOINT -->
+      <joint name="base_tip_joint" type="revolute">
+        <axis xyz="0 0 1"/>
+        <limit effort="1000.0" lower="-${90 * PI / 180}" upper="${90 * PI / 180}" velocity="0.5"/>
+        <origin xyz="0.17 -0.15 0.0" rpy="-${90 * PI / 180} 0 0" />  <!-- height is the clearance -->
+        <parent link="seventh_link"/>
+        <child link="tip_link"/>
+      </joint>
+      <transmission name="base_tip_joint_trans">
+        <type>transmission_interface/SimpleTransmission</type>
+        <joint name="base_tip_joint">
+          <hardwareInterface>EffortJointInterface</hardwareInterface>
+        </joint>
+        <actuator name="base_tip_joint_act">
+          <!-- This hardwareInterface element exists for compatibility
+               with ROS Hydro. -->
+          <hardwareInterface>EffortJointInterface</hardwareInterface>
+          <mechanicalReduction>1</mechanicalReduction>
+        </actuator>
+      </transmission>
+    <!-- TIP_LINK -->
+    <link name="tip_link">
+      <inertial>
+        <mass value="125.0" />
+        <origin xyz="0 0 0" />
+        <inertia  ixx="1.391" ixy="0.004"  ixz="0.0"  iyy="6.853"  iyz="0.0"  izz="6.125" />
+      </inertial>
+      <visual>
+         <origin xyz="0 0 0" rpy="0 0 0" />
+         <geometry>
+            <mesh filename="package://robospect_description/meshes/bases/robospect_head.STL" scale="1 1 1"/>
+         </geometry>
+         <material name="black">
+         </material>
+      </visual>
+      <collision>
+         <origin xyz="0 0 0" rpy="0 0 0 " />
+         <geometry>
+           <mesh filename="package://robospect_description/meshes/bases/robospect_head.STL" scale="1 1 1"/>
+         </geometry>
+      </collision>
+    </link>
   </xacro:macro>
 </robot>

Commit message: description: adjusting joints direction

File: robospect_description/urdf/bases/robospect_crane.urdf.xacro (robot description, xacro)
@@ -15,5 +15,6 @@
   <xacro:property name="joint_5_upper_limit" value="1.155"/>
   <xacro:property name="joint_5_pitch" value="1.05"/>
-  <xacro:property name="joint_6_pitch" value="-${joint_6_upper_limit/2.0}"/>
+  <!--xacro:property name="joint_6_pitch" value="-${joint_6_upper_limit/2.0}"/-->
+  <xacro:property name="joint_6_pitch" value="-1.032"/>
   <xacro:macro name="robospect_crane">
   <!-- FIRST_JOINT -->

Commit message: description: Crane transformations modified

File: robospect_description/urdf/bases/robospect_crane.urdf.xacro (robot description, xacro)
@@ -14,7 +14,8 @@
   <xacro:property name="joint_5_lower_limit" value="0.0"/>
   <xacro:property name="joint_5_upper_limit" value="1.155"/>
-  <xacro:property name="joint_5_pitch" value="1.05"/>
+  <xacro:property name="joint_5_pitch" value="0.6981"/>
   <!--xacro:property name="joint_6_pitch" value="-${joint_6_upper_limit/2.0}"/-->
-  <xacro:property name="joint_6_pitch" value="-1.032"/>
+  <xacro:property name="joint_6_pitch" value="1.5707"/>
+  <xacro:property name="joint_7_pitch" value="0.5061"/>
   <xacro:macro name="robospect_crane">
   <!-- FIRST_JOINT -->
@@ -32,6 +33,4 @@
       </joint>
       <actuator name="crane_first_joint_act">
-        <!-- This hardwareInterface element exists for compatibility
-             with ROS Hydro. -->
         <hardwareInterface>EffortJointInterface</hardwareInterface>
         <mechanicalReduction>1</mechanicalReduction>
@@ -68,6 +67,5 @@
       <axis xyz="0 0 1"/>
       <limit effort="1000.0" lower="${joint_2_lower_limit}" upper="${joint_2_upper_limit}" velocity="0.5"/>
-      <!--origin xyz="-0.28 0 1.25" rpy="0 0 0" /-->  <!-- height is the clearance -->
-      <origin xyz="-0.305 0 1.442" rpy="0 0 0" />  <!-- height is the clearance -->
+      <origin xyz="-0.305 0 1.442" rpy="0 0 0" />
       <parent link="first_link"/>
       <child link="second_link"/>
@@ -121,6 +119,4 @@
         </joint>
         <actuator name="crane_third_joint_act">
-          <!-- This hardwareInterface element exists for compatibility
-               with ROS Hydro. -->
           <hardwareInterface>EffortJointInterface</hardwareInterface>
           <mechanicalReduction>1</mechanicalReduction>
@@ -164,6 +160,4 @@
         </joint>
         <actuator name="crane_fourth_joint_act">
-          <!-- This hardwareInterface element exists for compatibility
-               with ROS Hydro. -->
           <hardwareInterface>EffortJointInterface</hardwareInterface>
           <mechanicalReduction>1</mechanicalReduction>
@@ -194,7 +188,7 @@
       <!-- FIFTH_JOINT -->
       <joint name="crane_fifth_joint" type="revolute">
-        <axis xyz="0 1 0"/>
+        <axis xyz="0 -1 0"/>
         <limit effort="1000.0" lower="${joint_5_lower_limit}" upper="${joint_5_upper_limit}" velocity="0.5"/>
-        <origin xyz="2.084 0 0.132" rpy="0 ${joint_5_pitch} 0" />
+        <origin xyz="2.084 0 0.132" rpy="0 ${PI/2 + joint_5_pitch} 0" />
         <parent link="fourth_link"/>
         <child link="fifth_link"/>
@@ -236,5 +230,5 @@
         <axis xyz="0 -1 0"/>
         <limit effort="1000.0" lower="${joint_6_lower_limit}" upper="${joint_6_upper_limit}" velocity="0.5"/>
-        <origin xyz="0.0 0.0 0.252" rpy="0 -${joint_5_pitch + joint_6_pitch} 0" />  <!-- height is the clearance -->
+        <origin xyz="0.0 0.0 0.252" rpy="0 ${PI/2.0} 0" />
         <parent link="fifth_link"/>
         <child link="sixth_link"/>
@@ -262,5 +256,5 @@
         <axis xyz="0 -1 0"/>
         <limit effort="1000.0" lower="${joint_6_lower_limit}" upper="${joint_6_upper_limit}" velocity="0.5"/>
-        <origin xyz="0.0 0.060 0.252" rpy="0 -${joint_5_pitch + joint_6_pitch} 0" />  <!-- height is the clearance -->
+        <origin xyz="0.0 0.060 0.252" rpy="0 0.0 0" />
         <parent link="fifth_link"/>
         <child link="crane_sixth_aux_1_link"/>
@@ -298,9 +292,9 @@
       </collision>
     </link>
-    <!-- SIXTH_AUX_JOINT 2 -->
+     <!-- SIXTH_AUX_JOINT 2 -->
     <joint name="crane_sixth_aux_2_joint" type="revolute">
         <axis xyz="0 -1 0"/>
         <limit effort="1000.0" lower="${joint_6_lower_limit}" upper="${joint_6_upper_limit}" velocity="0.5"/>
-        <origin xyz="0.0 -0.060 0.252" rpy="0 -${joint_5_pitch + joint_6_pitch} 0" />  <!-- height is the clearance -->
+        <origin xyz="0.0 -0.060 0.252" rpy="0 0 0" />  <!-- height is the clearance -->
         <parent link="fifth_link"/>
         <child link="crane_sixth_aux_2_link"/>
@@ -342,5 +336,5 @@
         <axis xyz="0 -1 0"/>
         <limit effort="1000.0" lower="${joint_6_lower_limit}" upper="${joint_6_upper_limit}" velocity="0.5"/>
-        <origin xyz="0.264 0.060 0.114" rpy="0 -${joint_5_pitch + joint_6_pitch} 0" />
+        <origin xyz="0.264 0.060 0.114" rpy="0 0 0" />
         <parent link="fifth_link"/>
         <child link="crane_sixth_aux_3_link"/>
@@ -382,5 +376,5 @@
         <axis xyz="0 -1 0"/>
         <limit effort="1000.0" lower="${joint_6_lower_limit}" upper="${joint_6_upper_limit}" velocity="0.5"/>
-        <origin xyz="0.264 -0.060 0.114" rpy="0 -${joint_5_pitch + joint_6_pitch} 0" />
+        <origin xyz="0.264 -0.060 0.114" rpy="0 0 0" />
         <parent link="fifth_link"/>
         <child link="crane_sixth_aux_4_link"/>
@@ -422,9 +416,8 @@
         <axis xyz="0 1 0"/>
         <limit effort="1000.0" lower="-1.57" upper="1.57" velocity="0.5"/>
-        <!--origin xyz="1.239 0 0" rpy="${90 * PI / 180} 0 0" /-->  <!-- height is the clearance -->
-        <origin xyz="1.239 0 0.0" rpy="0 ${joint_6_pitch} 0" />  <!-- height is the clearance -->
+        <origin xyz="0 0 1.239" rpy="0 ${PI + joint_7_pitch} 0" />
         <parent link="sixth_link"/>
         <child link="seventh_link"/>
-        <mimic joint="crane_sixth_joint" multiplier="1.0" offset="0.0"/> <!-- offset="-0.485" -->
+        <mimic joint="crane_sixth_joint" multiplier="1.0" offset="0.0"/>
       </joint>
       <transmission name="crane_seventh_joint_trans">
@@ -476,6 +469,4 @@
         </joint>
         <actuator name="crane_tip_joint_act">
-          <!-- This hardwareInterface element exists for compatibility
-               with ROS Hydro. -->
           <hardwareInterface>EffortJointInterface</hardwareInterface>
           <mechanicalReduction>1</mechanicalReduction>

Commit message: description: Correcting z coordinate of crane_second_link

File: robospect_description/urdf/bases/robospect_crane.urdf.xacro (robot description, xacro)
@@ -67,5 +67,5 @@
       <axis xyz="0 0 1"/>
       <limit effort="1000.0" lower="${joint_2_lower_limit}" upper="${joint_2_upper_limit}" velocity="0.5"/>
-      <origin xyz="-0.305 0 1.442" rpy="0 0 0" />
+      <origin xyz="-0.305 0 1.400" rpy="0 0 0" />
       <parent link="first_link"/>
       <child link="second_link"/>
