Commit message: Testing new configurations

File: robospect_description/robots/robospect_v2.urdf.xacro (robot description, xacro)
@@ -8,5 +8,5 @@
 	<xacro:include filename="$(find robospect_description)/urdf/bases/robospect_base.urdf.xacro" />
 	<!-- Import Robospect Crane -->
-	<xacro:include filename="$(find robospect_description)/urdf/bases/robospect_crane.urdf.xacro" />
+	<xacro:include filename="$(find robospect_description)/urdf/bases/robospect_crane_v2.urdf.xacro" />
 	<!-- Import Robospect Wheels -->
 	<xacro:include filename="$(find robospect_description)/urdf/wheels/standard_wheel.urdf.xacro" />
@@ -24,7 +24,5 @@
 	<!-- Genie base -->
 	<xacro:robospect_base name="robospect_base" publish_bf="true" />
-	<xacro:robospect_crane parent="base_link">
-		<origin xyz="-0.073 0 0.287" rpy="0 0 0" />
-	</xacro:robospect_crane>
+	<xacro:robospect_crane/>
 	<!-- Gazebo ros control pluggins -->
 	<xacro:ros_control/>
@@ -32,8 +30,17 @@
   <!-- Wheels -->
   <xacro:wheels parent="base_link"/>
+  <!--xacro:front_wheel lr_prefix="right" fr_prefix="rear"/>
+  <xacro:rear_wheel lr_prefix="left" fr_prefix="front">
+  <xacro:rear_wheel lr_prefix="right" fr_prefix="front"/-->
 	<!-- SENSORS -->
 	<xacro:sensor_imu name="imu" parent="base_link">
 		<origin xyz="0.0 0.0 0.170" rpy="0 0 0"/>
 	</xacro:sensor_imu>
+	<!--xacro:sensor_hokuyo_utm30lx name="sick_front" parent="base_link">
+		<origin xyz="1.058 0.0 0.0" rpy="0 0 0"/>
+	</xacro:sensor_hokuyo_utm30lx>
+	<xacro:sensor_hokuyo_utm30lx name="sick_rear" parent="base_link">
+		<origin xyz="-1.058 0.0 0.0" rpy="0 0 ${PI}"/>
+	</xacro:sensor_hokuyo_utm30lx!-->
 	<xacro:sensor_sick_s3000 name="sick_front" parent="base_link">
 		<origin xyz="1.058 0.0 0.0" rpy="0 0 0"/>
@@ -42,4 +49,9 @@
 		<origin xyz="-1.058 0.0 0.0" rpy="0 0 ${PI}"/>
 	</xacro:sensor_sick_s3000>
+<!--
+	<xacro:sensor_hokuyo_urg04lx name="hokuyo1" parent="base_link">
+		<origin xyz="-0.1 0.0 0.33" rpy="0 0 0"/>
+	</xacro:sensor_hokuyo_urg04lx>
+-->
 	<xacro:sensor_axis name="camera" parent="first_link">
 		<origin xyz="0.573 0 0.313" rpy="0 ${PI/180} 0"/>
@@ -47,5 +59,5 @@
 	<!-- NAV200 -->
     <joint name="nav200_laser_joint" type="fixed">
-	  <origin xyz="0.880 0.0 0.408" rpy="0 0 0"/>
+	  <origin xyz="0.9225 0.009 0.408" rpy="0 0 ${-PI/2}"/>
       <parent link="base_link"/>
       <child link="nav200_laser_link"/>
@@ -58,9 +70,9 @@
 		</inertial>
 	 </link>
-	<!--xacro:sensor_imu name="imu_crane" parent="tip_link">
+	<xacro:sensor_imu name="imu_crane" parent="tip_link">
 		<origin xyz="0.7 0.0 0.32" rpy="0 0 0"/>
-	</xacro:sensor_imu-->
+	</xacro:sensor_imu>
 	<!-- ARM UC3M -->
-    <!--joint name="arm_joint" type="fixed">
+    <joint name="arm_joint" type="fixed">
 	  <origin xyz="0.731 0.0 0.308" rpy="0 0 ${-PI/2}"/>
       <parent link="tip_link"/>
@@ -73,5 +85,5 @@
 			<inertia ixx="1e-6" ixy="0" ixz="0" iyy="1e-6" iyz="0" izz="1e-6" />
 		</inertial>
-	 </link-->
+	 </link>
 <!--
 	<xacro:sensor_asus_xtion_pro name="xtion_pro" parent="base_link">

File: robospect_description/urdf/bases/robospect_crane_v2.urdf.xacro (robot description, xacro)
@@ -15,10 +15,8 @@
   <xacro:property name="joint_5_lower_limit" value="0.0"/>
   <xacro:property name="joint_5_upper_limit" value="1.155"/>
-  <!--xacro:property name="joint_5_lower_limit" value="-0.4569"/>
-  <xacro:property name="joint_5_upper_limit" value="0.6981"/-->
-  <xacro:property name="joint_5_yaw" value="0.6981"/>
+  <xacro:property name="joint_5_pitch" value="0.6981"/>
   <!--xacro:property name="joint_6_pitch" value="-${joint_6_upper_limit/2.0}"/-->
   <xacro:property name="joint_6_pitch" value="1.5707"/>
-  <xacro:property name="joint_7_yaw" value="0.5061"/>
+  <xacro:property name="joint_7_pitch" value="0.5061"/>
   <xacro:macro name="robospect_crane" params="parent *origin">
   <!-- FIRST_JOINT -->
@@ -26,5 +24,4 @@
       <axis xyz="0 0 1"/>
       <limit effort="1000.0" lower="${joint_1_lower_limit}" upper="${joint_1_upper_limit}" velocity="0.5"/>
-      <!--origin xyz="-0.073 0 0.287" rpy="0 0 0" /-->
       <insert_block name="origin" />
       <parent link="${parent}"/>
@@ -67,5 +64,5 @@
     <material>Gazebo/White</material>
   </gazebo>
-	<!-- SECOND_JOINT -->
+  <!-- SECOND_JOINT -->
     <joint name="crane_second_joint" type="prismatic">
       <axis xyz="0 0 1"/>
@@ -110,26 +107,26 @@
   </link>
     <!-- THIRD_JOINT -->
-	<joint name="crane_third_joint" type="revolute">
-		<axis xyz="0 0 1"/>
-		<limit effort="100000.0" lower="${joint_3_lower_limit}" upper="${joint_3_upper_limit}" velocity="0.2"/>
-		<origin xyz="0 0 0" rpy="${PI/2.0} 0 0" />  <!-- height is the clearance -->
-		<parent link="second_link"/>
-		<child link="third_link"/>
-	</joint>
-	<transmission name="crane_third_joint_trans">
-		<type>transmission_interface/SimpleTransmission</type>
-		<joint name="crane_third_joint">
-		  <hardwareInterface>EffortJointInterface</hardwareInterface>
-		</joint>
-		<actuator name="crane_third_joint_act">
-		  <hardwareInterface>EffortJointInterface</hardwareInterface>
-		  <mechanicalReduction>1</mechanicalReduction>
-		</actuator>
-	</transmission>
+      <joint name="crane_third_joint" type="revolute">
+        <axis xyz="0 -1 0"/>
+        <limit effort="100000.0" lower="${joint_3_lower_limit}" upper="${joint_3_upper_limit}" velocity="0.2"/>
+        <origin xyz="0 0 0" rpy="0 0 0" />  <!-- height is the clearance -->
+        <parent link="second_link"/>
+        <child link="third_link"/>
+      </joint>
+      <transmission name="crane_third_joint_trans">
+        <type>transmission_interface/SimpleTransmission</type>
+        <joint name="crane_third_joint">
+          <hardwareInterface>EffortJointInterface</hardwareInterface>
+        </joint>
+        <actuator name="crane_third_joint_act">
+          <hardwareInterface>EffortJointInterface</hardwareInterface>
+          <mechanicalReduction>1</mechanicalReduction>
+        </actuator>
+      </transmission>
     <!-- THIRD_LINK -->
     <link name="third_link">
       <inertial>
         <mass value="2.0" />
-        <origin xyz="0 0 0" rpy="${PI/2.0} 0 0"/>
+        <origin xyz="0 0 0" />
         <inertia  ixx="1.391" ixy="0.004"  ixz="0.0"  iyy="6.853"  iyz="0.0"  izz="6.125" />
       </inertial>
@@ -143,5 +140,5 @@
       </visual>
       <collision>
-         <origin xyz="0 0 0" rpy="${PI/2.0} 0 0" />
+         <origin xyz="0 0 0" rpy="0 0 0 " />
          <geometry>
            <mesh filename="package://robospect_description/meshes/bases/robospect_third.dae" scale="1 1 1"/>
@@ -149,46 +146,32 @@
       </collision>
     </link>
-	<!-- FOURTH_JOINT -->
-	<joint name="crane_fourth_base_joint" type="fixed">
-		<axis xyz="0 0 1"/>
-		<!--origin xyz="2.8 0 0.04" rpy="0 0 0" /-->
-		<origin xyz="0.774 0 -0.087" rpy="0 ${PI/2} 0" />
-		<parent link="third_link"/>
-		<child link="fourth_base_link"/>
-	</joint>
-	<link name="fourth_base_link">
-      <inertial>
-        <mass value="0.0" />
-        <origin xyz="0 0 0" />
-        <inertia  ixx="0.0" ixy="0.0"  ixz="0.0"  iyy="0.0"  iyz="0.0"  izz="0.0" />
-      </inertial>
-	</link>
-	<joint name="crane_fourth_joint" type="prismatic">
-		<axis xyz="0 0 1"/>
-		<limit effort="1000.0" lower="${joint_4_lower_limit}" upper="${joint_4_upper_limit}" velocity="0.5"/>
-		<!--origin xyz="2.8 0 0.04" rpy="0 0 0" /-->
-		<origin xyz="0.0 0 0.0" rpy="0 0 -${PI/2}" />
-		<parent link="fourth_base_link"/>
-		<child link="fourth_link"/>
-	</joint>
-	<transmission name="crane_fourth_joint_trans">
-		<type>transmission_interface/SimpleTransmission</type>
-		<joint name="crane_fourth_joint">
-		  <hardwareInterface>EffortJointInterface</hardwareInterface>
-		</joint>
-		<actuator name="crane_fourth_joint_act">
-		  <hardwareInterface>EffortJointInterface</hardwareInterface>
-		  <mechanicalReduction>1</mechanicalReduction>
-		</actuator>
-	</transmission>
+    <!-- FOURTH_JOINT -->
+      <joint name="crane_fourth_joint" type="prismatic">
+        <axis xyz="1 0 0"/>
+        <limit effort="1000.0" lower="${joint_4_lower_limit}" upper="${joint_4_upper_limit}" velocity="0.5"/>
+        <!--origin xyz="2.8 0 0.04" rpy="0 0 0" /-->
+        <origin xyz="0.774 0 -0.087" rpy="0 0 0" />  <!-- height is the clearance -->
+        <parent link="third_link"/>
+        <child link="fourth_link"/>
+      </joint>
+      <transmission name="crane_fourth_joint_trans">
+        <type>transmission_interface/SimpleTransmission</type>
+        <joint name="crane_fourth_joint">
+          <hardwareInterface>EffortJointInterface</hardwareInterface>
+        </joint>
+        <actuator name="crane_fourth_joint_act">
+          <hardwareInterface>EffortJointInterface</hardwareInterface>
+          <mechanicalReduction>1</mechanicalReduction>
+        </actuator>
+      </transmission>
     <!-- FOURTH_LINK -->
     <link name="fourth_link">
       <inertial>
         <mass value="2.0" />
-        <origin xyz="0 0 0"/>
-        <inertia  ixx="1.391" ixy="0.004"  ixz="0.0"  iyy="6.853"  iyz="0.0"  izz="6.125" />
-      </inertial>
-      <visual>
-         <origin xyz="0 0 0" rpy="0 -${PI/2} 0" />
+        <origin xyz="0 0 0" />
+        <inertia  ixx="1.391" ixy="0.004"  ixz="0.0"  iyy="6.853"  iyz="0.0"  izz="6.125" />
+      </inertial>
+      <visual>
+         <origin xyz="0 0 0" rpy="0 0 0" />
          <geometry>
             <mesh filename="package://robospect_description/meshes/bases/robospect_fourth.dae" scale="1 1 1"/>
@@ -204,14 +187,13 @@
       </collision>
     </link>
-    <!-- FIFTH_JOINT -->
+      <!-- FIFTH_JOINT -->
       <joint name="crane_fifth_joint" type="revolute">
-        <axis xyz="0 0 -1"/>
-        <!--limit effort="1000.0" lower="${joint_5_lower_limit}" upper="${joint_5_upper_limit}" velocity="0.5"/-->
-        <limit effort="1000.0" lower="-${PI/2}" upper="${PI/2}" velocity="0.5"/>
-        <!--origin xyz="-0.132 0.0 2.084" rpy="-${PI/2.0} ${joint_5_yaw} 0" /-->
-        <origin xyz="-0.132 0.0 2.084" rpy="-${PI/2.0} ${joint_5_yaw - joint_5_upper_limit} 0" />
+        <axis xyz="0 -1 0"/>
+        <limit effort="1000.0" lower="${joint_5_lower_limit}" upper="${joint_5_upper_limit}" velocity="0.5"/>
+        <!--origin xyz="2.084 0 0.132" rpy="0 ${PI/2 + joint_5_pitch} 0" /-->
+        <origin xyz="2.084 0 0.132" rpy="0 ${PI/2 + joint_5_pitch} 0" />
         <parent link="fourth_link"/>
         <child link="fifth_link"/>
-        <mimic joint="crane_third_joint" multiplier="-1.0" offset="0.0"/>
+        <!--mimic joint="crane_third_joint" multiplier="-1.0" offset="0.0"/-->
       </joint>
       <transmission name="crane_fifth_joint_trans">
@@ -233,5 +215,5 @@
       </inertial>
       <visual>
-         <origin xyz="0 0 0" rpy="${PI/2.0} 0 0" />
+         <origin xyz="0 0 0" rpy="0 0 0" />
          <geometry>
             <mesh filename="package://robospect_description/meshes/bases/robospect_fifth.dae" scale="1 1 1"/>
@@ -241,6 +223,5 @@
       </visual>
       <collision>
-         <!--origin xyz="0 0 0" rpy="${PI/2.0} 0 ${joint_5_yaw}" /-->
-         <origin xyz="0 0 0" rpy="${PI/2.0} 0 0" />
+         <origin xyz="0 0 0" rpy="0 0 0 " />
          <geometry>
            <mesh filename="package://robospect_description/meshes/bases/robospect_fifth.dae" scale="1 1 1"/>
@@ -248,11 +229,9 @@
       </collision>
     </link>
-	<!-- SIXTH_JOINT -->
+     <!-- SIXTH_JOINT -->
       <joint name="crane_sixth_joint" type="revolute">
-        <axis xyz="0 0 -1"/>
+        <axis xyz="0 -1 0"/>
         <limit effort="1000.0" lower="${joint_6_lower_limit}" upper="${joint_6_upper_limit}" velocity="0.5"/>
-        <!--origin xyz="0.0 0.0 0.252" rpy="0 ${PI/2.0} 0" /-->
-        <!--origin xyz="0 -0.252 0" rpy="0 0 -${PI/2}" /-->
-        <origin xyz="0 -0.252 0" rpy="0 0 0" />
+        <origin xyz="0.0 0.0 0.252" rpy="0 ${PI/2.0} 0" />
         <parent link="fifth_link"/>
         <child link="sixth_link"/>
@@ -276,9 +255,9 @@
       </inertial>
     </link>
-    <!-- SEVENTH_JOINT -->
+     <!-- SEVENTH_JOINT -->
       <joint name="crane_seventh_joint" type="revolute">
-        <axis xyz="0 0 1"/>
+        <axis xyz="0 1 0"/>
         <limit effort="1000.0" lower="-1.57" upper="1.57" velocity="0.5"/>
-        <origin xyz="1.239 0 0" rpy="0 0 ${joint_7_yaw -PI/2.0}" />
+        <origin xyz="0 0 1.239" rpy="0 ${PI + joint_7_pitch} 0" />
         <parent link="sixth_link"/>
         <child link="seventh_link"/>
@@ -291,4 +270,6 @@
         </joint>
         <actuator name="crane_seventh_joint_act">
+          <!-- This hardwareInterface element exists for compatibility
+               with ROS Hydro. -->
           <hardwareInterface>EffortJointInterface</hardwareInterface>
           <mechanicalReduction>1</mechanicalReduction>
@@ -303,5 +284,5 @@
       </inertial>
       <visual>
-         <origin xyz="0 0 0" rpy="${PI/2.0} 0 0" />
+         <origin xyz="0 0 0" rpy="0 0 0" />
          <geometry>
             <mesh filename="package://robospect_description/meshes/bases/robospect_seventh.dae" scale="1 1 1"/>
@@ -311,5 +292,5 @@
       </visual>
       <collision>
-         <origin xyz="0 0 0" rpy="${PI/2.0} 0 0 " />
+         <origin xyz="0 0 0" rpy="0 0 0 " />
          <geometry>
            <mesh filename="package://robospect_description/meshes/bases/robospect_seventh.dae" scale="1 1 1"/>
@@ -317,10 +298,9 @@
       </collision>
     </link>
-     <!-- TIP_JOINT -->
+        <!-- TIP_JOINT -->
       <joint name="crane_tip_joint" type="revolute">
         <axis xyz="0 0 1"/>
         <limit effort="1000.0" lower="-${90 * PI / 180}" upper="${90 * PI / 180}" velocity="0.5"/>
-        <!--origin xyz="0.164 0.0 -0.155" rpy="0 0 0" /-->
-        <origin xyz="0.164 0.0 0.0" rpy="${PI/2.0} 0 0" />
+        <origin xyz="0.164 0.0 -0.155" rpy="0 0 0" />
         <parent link="seventh_link"/>
         <child link="tip_link"/>
@@ -344,5 +324,5 @@
       </inertial>
       <visual>
-         <origin xyz="0 0 -0.155" rpy="0 0 0" />
+         <origin xyz="0 0 0" rpy="0 0 0" />
          <geometry>
             <mesh filename="package://robospect_description/meshes/bases/robospect_head.dae" scale="1 1 1"/>
