Commit message: Major modifications in the base

File: robospect_description/robots/robospect.urdf.xacro (robot description, xacro)
@@ -5,7 +5,9 @@
 	<!-- ***************** -->
 	<!-- First we import all posible elements defined in the urdf.xacro files. All these elements are defined as macro:xacros -->
-	<!-- Import Robotnik CAR base elements -->
+	<!-- Import Robospect Base -->
 	<xacro:include filename="$(find robospect_description)/urdf/bases/robospect_base.urdf.xacro" />
-	<!-- Import Robotnik CAR wheels -->
+	<!-- Import Robospect Crane -->
+	<xacro:include filename="$(find robospect_description)/urdf/bases/robospect_base.urdf.xacro" />
+	<!-- Import Robospect Wheels -->
 	<xacro:include filename="$(find robospect_description)/urdf/wheels/suspension_wheel.urdf.xacro" />
 	<!-- Import all available sensors -->
@@ -19,26 +21,22 @@
 	<xacro:property name="wheel_offset_y" value="0.75" />
 	<xacro:property name="wheel_offset_z" value="0.0" />
-	<!-- Flag to select the high or low quality model -->
-	<xacro:property name="hq" value="true" />
 	<!-- *************** -->
 	<!-- Robots Elements -->
 	<!-- *************** -->
 	<!-- Here we create the robot elements using the xacro:macros imported at the beggining of this file -->
-	<!-- Summit XL base -->
-	<xacro:robospect_base name="robospect" publish_bf="true" hq="${hq}" />
+	<!-- Genie base -->
+	<xacro:robospect_base name="robospect" publish_bf="true" />
 	<!-- Gazebo ros control pluggins -->
 	<xacro:ros_control/>
-	<!-- Gazebo skid steering pluggins -->
-	<!-- xacro:skid_steering broadcastOdomTF="1"/ -->
 	<!-- WHEELS -->
   <!-- Wheels -->
-  <xacro:front_wheel lr_prefix="left" fr_prefix="front"
-                     lr_reflect="1" fr_reflect="1"/>
-  <xacro:front_wheel lr_prefix="right" fr_prefix="front"
-                     lr_reflect="-1" fr_reflect="1"/>
-  <xacro:rear_wheel lr_prefix="left" fr_prefix="rear"
-                    lr_reflect="1" fr_reflect="-1"/>
-  <xacro:rear_wheel lr_prefix="right" fr_prefix="rear"
-                    lr_reflect="-1" fr_reflect="-1"/>
+  <xacro:front_wheel lr_prefix="left" fr_prefix="rear"
+                     lr_reflect="1" fr_reflect="-1"/>
+  <xacro:front_wheel lr_prefix="right" fr_prefix="rear"
+                     lr_reflect="-1" fr_reflect="-1"/>
+  <xacro:rear_wheel lr_prefix="left" fr_prefix="front"
+                    lr_reflect="1" fr_reflect="1"/>
+  <xacro:rear_wheel lr_prefix="right" fr_prefix="front"
+                    lr_reflect="-1" fr_reflect="1"/>
 	<!-- SENSORS -->
 	<xacro:sensor_imu name="imu" parent="base_link">
@@ -54,5 +52,5 @@
 -->
 	<xacro:sensor_axis name="camera" parent="base_link">
-		<origin xyz="0.19 0 0.17" rpy="0 ${15*PI/180} 0"/>
+		<origin xyz="0.9 0 0.37" rpy="0 ${PI/180} 0"/>
 	</xacro:sensor_axis>
 <!--

File: robospect_description/urdf/bases/robospect_base.urdf.xacro (robot description, xacro)
@@ -2,5 +2,5 @@
 <robot name="robospect" xmlns:xacro="http://www.ros.org/wiki/xacro">
   <xacro:include filename="$(find robospect_description)/urdf/bases/robospect_base.gazebo.xacro" />
-  <xacro:macro name="robospect_base" params="name publish_bf hq">
+  <xacro:macro name="robospect_base" params="name publish_bf">
   <!-- Robot mechanical and motor parameters -->
   <xacro:property name="PI" value="3.1415926535897931"/>
@@ -25,5 +25,5 @@
     </link>
     <joint name="base_footprint_joint" type="fixed">
-      <origin xyz="0 0 0.235" rpy="0 0 0" />  <!-- height is the clearance -->
+      <origin xyz="0 0 0.296166007" rpy="0 0 0" />  <!-- height is the clearance -->
       <parent link="base_footprint"/>
       <child link="base_link" />
@@ -38,21 +38,14 @@
     </inertial>
     <visual>
-       <origin xyz="0 0 0" rpy="0 0 0" />
-       <xacro:if value="${hq}">
+       <origin xyz="0 0 -0.17" rpy="0 0 ${PI/2}" />
        <geometry>
-	     <mesh filename="package://robospect_description/meshes/bases/robospect_chassis.stl"/>
+	       <mesh filename="package://robospect_description/meshes/bases/robospect_chassis.stl"/>
        </geometry>
-       </xacro:if>
-       <xacro:unless value="${hq}">
-       <geometry>
-	     <mesh filename="package://robospect_description/meshes/bases/robospect_chassis.stl"/>
-       </geometry>
-       </xacro:unless>
-       <material name="darkgrey">
-         <color rgba="0.1 0.1 0.1 1"/>
+       <material name="blue">
+         <color rgba="0.0 0.4 0.9 1.0"/>
        </material>
     </visual>
     <collision>
-       <origin xyz="0 0 0" rpy="0 0 0 " />
+       <origin xyz="0 0 -0.17" rpy="0 0 ${PI/2}" />
        <geometry>
          <mesh filename="package://robospect_description/meshes/bases/robospect_chassis.stl"/>

File: robospect_description/urdf/wheels/suspension_wheel.urdf.xacro (robot description, xacro)
@@ -7,13 +7,13 @@
        axle_length. -->
   <xacro:property name="hub_dia" value="0.235"/>
-  <xacro:property name="tire_dia" value="0.470"/>
+  <xacro:property name="tire_dia" value="0.592332013"/>
   <xacro:property name="tire_width" value="0.2"/>
   <xacro:property name="hex_hub_depth" value="0.120"/> <!-- or +0.072 -->
-  <xacro:property name="wheel_mass" value="8.0"/>   <!-- check -->
+  <xacro:property name="wheel_mass" value="15.0"/>   <!-- check -->
   <!-- hex_hub_dist is the distance between left and right hex hubs when
        the shock absorbers are fully extended. axle_length is the distance
        from a U joint to the corresponding hex hub. wheel_travel is the
        vertical wheel travel. -->
-  <xacro:property name="wheelbase" value="1.650"/>
+  <xacro:property name="wheelbase" value="1.645143603"/>
   <xacro:property name="hex_hub_dist" value="0.900"/>  <!-- 1.127 0.742 check -->
   <xacro:property name="axle_length" value="0.120"/>
@@ -130,5 +130,5 @@
     </transmission>
     <gazebo reference="${lr_prefix}_${fr_prefix}_axle_carrier">
-      <material>Gazebo/Black</material>
+      <material>Gazebo/White</material>
     </gazebo>
     <link name="${lr_prefix}_${fr_prefix}_wheel">
@@ -155,5 +155,5 @@
     </link>
     <gazebo reference="${lr_prefix}_${fr_prefix}_wheel">
-      <material>Gazebo/Black</material>
+      <material>Gazebo/White</material>
     </gazebo>
   </xacro:macro>
@@ -200,5 +200,5 @@
     </transmission>
     <gazebo reference="${lr_prefix}_steering_link">
-      <material>Gazebo/Black</material>
+      <material>Gazebo/White</material>
     </gazebo>
     <xacro:wheel lr_prefix="${lr_prefix}" fr_prefix="${fr_prefix}"

Commit message: First two joints of the crane added.

File: robospect_description/robots/robospect.urdf.xacro (robot description, xacro)
@@ -8,5 +8,5 @@
 	<xacro:include filename="$(find robospect_description)/urdf/bases/robospect_base.urdf.xacro" />
 	<!-- Import Robospect Crane -->
-	<xacro:include filename="$(find robospect_description)/urdf/bases/robospect_base.urdf.xacro" />
+	<xacro:include filename="$(find robospect_description)/urdf/bases/robospect_crane.urdf.xacro" />
 	<!-- Import Robospect Wheels -->
 	<xacro:include filename="$(find robospect_description)/urdf/wheels/suspension_wheel.urdf.xacro" />
@@ -26,5 +26,6 @@
 	<!-- Here we create the robot elements using the xacro:macros imported at the beggining of this file -->
 	<!-- Genie base -->
-	<xacro:robospect_base name="robospect" publish_bf="true" />
+	<xacro:robospect_base name="robospect_base" publish_bf="true" />
+	<xacro:robospect_crane/>
 	<!-- Gazebo ros control pluggins -->
 	<xacro:ros_control/>

File: robospect_description/urdf/bases/robospect_base.urdf.xacro (robot description, xacro)
@@ -38,7 +38,7 @@
     </inertial>
     <visual>
-       <origin xyz="0 0 -0.17" rpy="0 0 ${PI/2}" />
+       <origin xyz="0 0 0" rpy="0 0 0" />
        <geometry>
-	       <mesh filename="package://robospect_description/meshes/bases/robospect_chassis.stl"/>
+	       <mesh filename="package://robospect_description/meshes/bases/robospect_base_chassis.STL"/>
        </geometry>
        <material name="blue">
@@ -47,7 +47,7 @@
     </visual>
     <collision>
-       <origin xyz="0 0 -0.17" rpy="0 0 ${PI/2}" />
+       <origin xyz="0 0 0" rpy="0 0 0" />
        <geometry>
-         <mesh filename="package://robospect_description/meshes/bases/robospect_chassis.stl"/>
+         <mesh filename="package://robospect_description/meshes/bases/robospect_base_chassis.STL"/>
        </geometry>
     </collision>

File: robospect_description/urdf/bases/robospect_crane.urdf.xacro (robot description, xacro)
@@ -3,4 +3,24 @@
   <!-- <xacro:include filename="$(find robospect_description)/urdf/bases/robospect_crane.gazebo.xacro" /> -->
   <xacro:macro name="robospect_crane">
+  <!-- FIRST_JOINT -->
+    <joint name="base_first_joint" type="revolute">
+      <axis xyz="0 0 1"/>
+      <limit effort="1000.0" lower="-${90 * PI / 180}" upper="${90 * PI / 180}" velocity="0.5"/>
+      <origin xyz="-0.046851 0 0.3" rpy="0 0 0" />  <!-- height is the clearance -->
+      <parent link="base_link"/>
+      <child link="first_link"/>
+    </joint>
+    <transmission name="base_first_joint_trans">
+      <type>transmission_interface/SimpleTransmission</type>
+      <joint name="base_first_joint">
+        <hardwareInterface>EffortJointInterface</hardwareInterface>
+      </joint>
+      <actuator name="base_first_joint_act">
+        <!-- This hardwareInterface element exists for compatibility
+             with ROS Hydro. -->
+        <hardwareInterface>EffortJointInterface</hardwareInterface>
+        <mechanicalReduction>1</mechanicalReduction>
+      </actuator>
+    </transmission>
   <!-- FIRST_LINK -->
   <link name="first_link">
@@ -13,8 +33,8 @@
        <origin xyz="0 0 0" rpy="0 0 0" />
        <geometry>
-	        <mesh filename="package://robospect_description/meshes/bases/robospect_crane_1.stl"/>
+	        <mesh filename="package://robospect_description/meshes/bases/robospect_first.STL" scale="1 1 1"/>
        </geometry>
-       <material name="blue">
-          <color rgba="0.1 0.2 0.8 1"/>
+       <material name="grey">
+          <color rgba="0.8 0.8 0.8 0.95"/>
        </material>
     </visual>
@@ -22,5 +42,47 @@
        <origin xyz="0 0 0" rpy="0 0 0 " />
        <geometry>
-         <mesh filename="package://robospect_description/meshes/bases/robospect_crane_1.stl"/>
+         <mesh filename="package://robospect_description/meshes/bases/robospect_first.STL" scale="1 1 1"/>
+       </geometry>
+    </collision>
+  </link>
+  <!-- SECOND_JOINT -->
+    <joint name="base_second_joint" type="prismatic">
+      <axis xyz="0 0 1"/>
+      <limit effort="1000.0" lower="0.0" upper="2.0" velocity="0.5"/>
+      <origin xyz="-0.3 0 1.25" rpy="0 0 0" />  <!-- height is the clearance -->
+      <parent link="first_link"/>
+      <child link="second_link"/>
+    </joint>
+    <transmission name="base_second_joint_trans">
+      <type>transmission_interface/SimpleTransmission</type>
+      <joint name="base_second_joint">
+        <hardwareInterface>EffortJointInterface</hardwareInterface>
+      </joint>
+      <actuator name="base_second_joint_act">
+        <!-- This hardwareInterface element exists for compatibility
+             with ROS Hydro. -->
+        <hardwareInterface>EffortJointInterface</hardwareInterface>
+        <mechanicalReduction>1</mechanicalReduction>
+      </actuator>
+    </transmission>
+  <!-- SECOND_LINK -->
+  <link name="second_link">
+    <inertial>
+      <mass value="125.0" />
+      <origin xyz="0 0 0" />
+      <inertia  ixx="1.391" ixy="0.004"  ixz="0.0"  iyy="6.853"  iyz="0.0"  izz="6.125" />
+    </inertial>
+    <visual>
+       <origin xyz="0 0 0" rpy="0 0 0" />
+       <geometry>
+	        <mesh filename="package://robospect_description/meshes/bases/robospect_second.STL" scale="1 1 1"/>
+       </geometry>
+       <material name="blue">
+       </material>
+    </visual>
+    <collision>
+       <origin xyz="0 0 0" rpy="0 0 0 " />
+       <geometry>
+         <mesh filename="package://robospect_description/meshes/bases/robospect_second.STL" scale="1 1 1"/>
        </geometry>
     </collision>

File: robospect_description/urdf/wheels/suspension_wheel.urdf.xacro (robot description, xacro)
@@ -7,5 +7,5 @@
        axle_length. -->
   <xacro:property name="hub_dia" value="0.235"/>
-  <xacro:property name="tire_dia" value="0.592332013"/>
+  <xacro:property name="tire_dia" value="0.56"/>
   <xacro:property name="tire_width" value="0.2"/>
   <xacro:property name="hex_hub_depth" value="0.120"/> <!-- or +0.072 -->
@@ -15,5 +15,5 @@
        from a U joint to the corresponding hex hub. wheel_travel is the
        vertical wheel travel. -->
-  <xacro:property name="wheelbase" value="1.645143603"/>
+  <xacro:property name="wheelbase" value="1.6"/>
   <xacro:property name="hex_hub_dist" value="0.900"/>  <!-- 1.127 0.742 check -->
   <xacro:property name="axle_length" value="0.120"/>

Commit message: Adding new wheels system to the URDF and testing new params

File: robospect_description/robots/robospect.urdf.xacro (robot description, xacro)
@@ -10,5 +10,5 @@
 	<xacro:include filename="$(find robospect_description)/urdf/bases/robospect_crane.urdf.xacro" />
 	<!-- Import Robospect Wheels -->
-	<xacro:include filename="$(find robospect_description)/urdf/wheels/suspension_wheel.urdf.xacro" />
+	<xacro:include filename="$(find robospect_description)/urdf/wheels/standard_wheel.urdf.xacro" />
 	<!-- Import all available sensors -->
 	<xacro:include filename="$(find robotnik_sensors)/urdf/all_sensors.urdf.xacro" />
@@ -18,7 +18,4 @@
 	<xacro:property name="PI" value="3.1415926535897931"/>
 	<!-- Wheel parameters -->
-	<xacro:property name="wheel_offset_x" value="1.0" />    <!-- x,y,z in translation from base_link to the center of the wheel -->
-	<xacro:property name="wheel_offset_y" value="0.75" />
-	<xacro:property name="wheel_offset_z" value="0.0" />
 	<!-- *************** -->
 	<!-- Robots Elements -->
@@ -32,12 +29,8 @@
 	<!-- WHEELS -->
   <!-- Wheels -->
-  <xacro:front_wheel lr_prefix="left" fr_prefix="rear"
-                     lr_reflect="1" fr_reflect="-1"/>
-  <xacro:front_wheel lr_prefix="right" fr_prefix="rear"
-                     lr_reflect="-1" fr_reflect="-1"/>
-  <xacro:rear_wheel lr_prefix="left" fr_prefix="front"
-                    lr_reflect="1" fr_reflect="1"/>
-  <xacro:rear_wheel lr_prefix="right" fr_prefix="front"
-                    lr_reflect="-1" fr_reflect="1"/>
+  <xacro:wheels parent="base_link"/>
+  <!--xacro:front_wheel lr_prefix="right" fr_prefix="rear"/>
+  <xacro:rear_wheel lr_prefix="left" fr_prefix="front">
+  <xacro:rear_wheel lr_prefix="right" fr_prefix="front"/-->
 	<!-- SENSORS -->
 	<xacro:sensor_imu name="imu" parent="base_link">

File: robospect_description/urdf/bases/robospect_base.urdf.xacro (robot description, xacro)
@@ -32,5 +32,5 @@
   <link name="base_link">
     <inertial>
-      <mass value="50.0" />
+      <mass value="200.0" />
       <origin xyz="0 0 0" />
       <inertia  ixx="1.391" ixy="0.004"  ixz="0.0"  iyy="6.853"  iyz="0.0"  izz="6.125" />

File: robospect_description/urdf/bases/robospect_crane.urdf.xacro (robot description, xacro)
@@ -260,8 +260,8 @@
     </link>
     <!-- SIXTH_AUX_JOINT -->
-      <joint name="crane_sixth_aux_joint" type="revolute">
+      <!--joint name="crane_sixth_aux_joint" type="revolute">
         <axis xyz="0 1 0"/>
         <limit effort="1000.0" lower="0" upper="1.3" velocity="0.5"/>
-        <origin xyz="0.1177 0 -0.26422" rpy="0 0 0" />  <!-- height is the clearance -->
+        <origin xyz="0.1177 0 -0.26422" rpy="0 0 0" />
         <parent link="fifth_link"/>
         <child link="sixth_aux_link"/>
@@ -270,15 +270,12 @@
       <transmission name="crane_sixth_aux_joint_trans">
         <type>transmission_interface/SimpleTransmission</type>
-        <joint name="crane_sixth_joint">
+        <joint name="crane_sixth_aux_joint">
           <hardwareInterface>EffortJointInterface</hardwareInterface>
         </joint>
         <actuator name="crane_sixth_aux_joint_act">
-          <!-- This hardwareInterface element exists for compatibility
-               with ROS Hydro. -->
-          <hardwareInterface>EffortJointInterface</hardwareInterface>
-          <mechanicalReduction>1</mechanicalReduction>
-        </actuator>
-      </transmission>
-    <!-- SIXTH_AUX_LINK -->
+          <hardwareInterface>EffortJointInterface</hardwareInterface>
+          <mechanicalReduction>1</mechanicalReduction>
+        </actuator>
+      </transmission>
     <link name="sixth_aux_link">
       <inertial>
@@ -301,5 +298,5 @@
          </geometry>
       </collision>
-    </link>
+    </link-->
     <!-- SEVENTH_JOINT -->
       <joint name="crane_seventh_joint" type="revolute">

Commit message: Added laser to base

File: robospect_description/robots/robospect.urdf.xacro (robot description, xacro)
@@ -37,7 +37,7 @@
 		<origin xyz="0.0 0.0 0.170" rpy="0 0 0"/>
 	</xacro:sensor_imu>
-	<!--xacro:sensor_hokuyo_utm30lx name="hokuyo" parent="base_link">
-		<origin xyz="0.0 0.0 0.33" rpy="0 0 0"/>
-	</xacro:sensor_hokuyo_utm30lx -->
+	<xacro:sensor_hokuyo_utm30lx name="hokuyo" parent="base_link">
+		<origin xyz="1 0.0 0.25" rpy="0 0 0"/>
+	</xacro:sensor_hokuyo_utm30lx>
 <!--
 	<xacro:sensor_hokuyo_urg04lx name="hokuyo1" parent="base_link">
