Commit message: robospect_description: setting the correct location for sick lasers

File: robospect_description/robots/robospect.urdf.xacro (robot description, xacro)
@@ -37,6 +37,9 @@
 		<origin xyz="0.0 0.0 0.170" rpy="0 0 0"/>
 	</xacro:sensor_imu>
-	<xacro:sensor_hokuyo_utm30lx name="hokuyo" parent="base_link">
-		<origin xyz="1 0.0 0.25" rpy="0 0 0"/>
+	<xacro:sensor_hokuyo_utm30lx name="sick_front" parent="base_link">
+		<origin xyz="1.058 0.0 0.0" rpy="0 0 0"/>
+	</xacro:sensor_hokuyo_utm30lx>
+	<xacro:sensor_hokuyo_utm30lx name="sick_rear" parent="base_link">
+		<origin xyz="-1.058 0.0 0.0" rpy="0 0 ${PI}"/>
 	</xacro:sensor_hokuyo_utm30lx>
 <!--
@@ -46,6 +49,19 @@
 -->
 	<xacro:sensor_axis name="camera" parent="base_link">
-		<origin xyz="0.9 0 0.37" rpy="0 ${PI/180} 0"/>
+		<origin xyz="0.5 0 0.6" rpy="0 ${PI/180} 0"/>
 	</xacro:sensor_axis>
+	<!-- NAV200 -->
+    <joint name="nav200_laser_joint" type="fixed">
+	  <origin xyz="0.9225 0.009 0.408" rpy="0 0 ${-PI/2}"/>
+      <parent link="base_link"/>
+      <child link="nav200_laser_link"/>
+	 </joint>
+	 <link name="nav200_laser_link">
+		<inertial>
+			<mass value="1e-5" />
+			<origin xyz="0 0 0" rpy="0 0 0"/>
+			<inertia ixx="1e-6" ixy="0" ixz="0" iyy="1e-6" iyz="0" izz="1e-6" />
+		</inertial>
+	 </link>
 <!--
 	<xacro:sensor_asus_xtion_pro name="xtion_pro" parent="base_link">

File: robospect_description/urdf/wheels/standard_wheel.urdf.xacro (robot description, xacro)
@@ -1,7 +1,12 @@
 <?xml version="1.0"?>
 <robot name="wheel" xmlns:xacro="http://www.ros.org/wiki/xacro">
-  <xacro:property name="wheel_offset_x" value="0.800" />    <!-- x,y,z in base_footprint CS -->
-  <xacro:property name="wheel_offset_y" value="0.56" />
+  <xacro:property name="wheel_offset_x" value="0.7725" />    <!-- x,y,z in base_footprint CS -->
+  <xacro:property name="wheel_offset_y" value="0.5025" />
   <xacro:property name="wheel_offset_z" value="0.0" />
+  <xacro:property name="steering_offset_x" value="0.7725" />    <!-- x,y,z in base_footprint CS -->
+  <xacro:property name="steering_offset_y" value="0.365" />
+  <xacro:property name="steering_offset_z" value="0.0" />
+  <xacro:property name="wheel_to_steering" value="0.11" />
+  <xacro:property name="wheel_width" value="0.175" />
   <xacro:property name="wheel_joint_damping" value="1.0" />
   <xacro:property name="wheel_joint_friction" value="1.0" />
@@ -28,13 +33,13 @@
   <xacro:property name="axle_vel_limit" value="39.02"/>
   <!-- The "wheel" macro defines an axle carrier, axle, and wheel. -->
-  <xacro:macro name="traction_wheel" params="parent prefix y_reflect x_reflect roll_reflect yaw_reflect">
+  <xacro:macro name="traction_wheel" params="parent prefix y_reflect x_reflect roll_reflect yaw_reflect x_pos y_pos z_pos x_link_offset y_link_offset z_link_offset">
 	<link name="${prefix}_wheel_link">
 	<inertial>
       <mass value="10" />
-      <origin xyz="0 0 0" />
+      <origin xyz="${x_link_offset} ${y_link_offset} ${z_link_offset}" />
       <inertia  ixx="0.01" ixy="0.0"  ixz="0.0"  iyy="0.01"  iyz="0.0"  izz="0.01" />
     </inertial>
       <visual>
-        <origin xyz="0 0 0"/>
+        <origin xyz="${x_link_offset} ${y_link_offset} ${z_link_offset}"/>
         <geometry>
           <mesh filename="package://robospect_description/meshes/wheels/robospect_wheel_l.STL" scale="1 1 1"/>
@@ -44,5 +49,5 @@
       </visual>
       <collision>
-        <origin xyz="0 0 0"/>
+        <origin xyz="${x_link_offset} ${y_link_offset} ${z_link_offset}"/>
         <geometry>
           <mesh filename="package://robospect_description/meshes/wheels/robospect_wheel_l.STL" scale="1 1 1"/>
@@ -53,5 +58,5 @@
       <parent link="${parent}"/>
       <child link="${prefix}_wheel_link"/>
-      <origin xyz="${x_reflect * wheel_offset_x} ${y_reflect * wheel_offset_y} ${wheel_offset_z}" rpy="${-roll_reflect * degrees_90} 0 ${yaw_reflect * degrees_180}"/>
+      <origin xyz="${x_reflect * x_pos} ${y_reflect * y_pos} ${z_pos}" rpy="${-roll_reflect * degrees_90} 0 ${yaw_reflect * degrees_180}"/>
       <axis xyz="0 0 ${yaw_reflect}"/>
       <limit effort="${axle_eff_limit}" velocity="${axle_vel_limit}"/>
@@ -77,5 +82,5 @@
     </gazebo>
   </xacro:macro>
-  <xacro:macro name="steering_wheel" params="parent prefix y_reflect x_reflect roll_reflect yaw_reflect">
+  <xacro:macro name="steering_wheel" params="parent prefix y_reflect x_reflect roll_reflect yaw_reflect x_pos y_pos z_pos">
 	<link name="${prefix}_steering_link">
 		<inertial>
@@ -86,5 +91,5 @@
     </link>
     <joint name="${prefix}_steering_joint" type="revolute">
-	  <origin xyz="${x_reflect * wheel_offset_x} ${y_reflect * wheel_offset_y} 0"/>
+	  <origin xyz="${x_reflect * x_pos} ${y_reflect * y_pos} ${z_pos}"/>
       <parent link="${parent}"/>
       <child link="${prefix}_steering_link"/>
@@ -105,12 +110,12 @@
     <gazebo reference="${prefix}_steering_link">
     </gazebo>
-    <xacro:traction_wheel prefix="${prefix}" parent="${prefix}_steering_link" x_reflect="0" y_reflect="0" yaw_reflect="${yaw_reflect}" roll_reflect="${roll_reflect}"/>
+    <xacro:traction_wheel prefix="${prefix}" parent="${prefix}_steering_link" x_reflect="0" y_reflect="${y_reflect}" yaw_reflect="${yaw_reflect}" roll_reflect="${roll_reflect}" x_pos="0.0" y_pos="${wheel_to_steering}" z_pos="0.0" x_link_offset="0.0" y_link_offset="0.0" z_link_offset="${-wheel_width/2.0}"/>
   </xacro:macro>
   <xacro:macro name="wheels"
                params="parent">
-    <xacro:traction_wheel prefix="left_front" parent="${parent}" x_reflect="1" y_reflect="1" yaw_reflect="1" roll_reflect="1"/>
-    <xacro:traction_wheel prefix="right_front" parent="${parent}" x_reflect="1" y_reflect="-1" yaw_reflect="-1" roll_reflect="-1"/>
-    <xacro:steering_wheel prefix="left_rear" parent="${parent}" x_reflect="-1" y_reflect="1" yaw_reflect="1" roll_reflect="1"/>
-    <xacro:steering_wheel prefix="right_rear" parent="${parent}" x_reflect="-1" y_reflect="-1" yaw_reflect="-1" roll_reflect="-1"/>
+    <xacro:traction_wheel prefix="left_front" parent="${parent}" x_reflect="1" y_reflect="1" yaw_reflect="1" roll_reflect="1" x_pos="${wheel_offset_x}" y_pos="${wheel_offset_y}" z_pos="0.0" x_link_offset="0.0" y_link_offset="0.0" z_link_offset="${-wheel_width/2.0}"/>
+    <xacro:traction_wheel prefix="right_front" parent="${parent}" x_reflect="1" y_reflect="-1" yaw_reflect="-1" roll_reflect="-1" x_pos="${wheel_offset_x}" y_pos="${wheel_offset_y}" z_pos="0.0" x_link_offset="0.0" y_link_offset="0.0" z_link_offset="${-wheel_width/2.0}"/>
+    <xacro:steering_wheel prefix="left_rear" parent="${parent}" x_reflect="-1" y_reflect="1" yaw_reflect="1" roll_reflect="1" x_pos="${steering_offset_x}" y_pos="${steering_offset_y}" z_pos="0.0"/>
+    <xacro:steering_wheel prefix="right_rear" parent="${parent}" x_reflect="-1" y_reflect="-1" yaw_reflect="-1" roll_reflect="-1" x_pos="${steering_offset_x}" y_pos="${steering_offset_y}" z_pos="0.0"/>
   </xacro:macro>
  <!--

Commit message: Adding new link for the IMU located on the crane tip. Changing pad topic name

File: robospect_description/robots/robospect.urdf.xacro (robot description, xacro)
@@ -64,4 +64,7 @@
 		</inertial>
 	 </link>
+	<xacro:sensor_imu name="imu_crane" parent="tip_link">
+		<origin xyz="0.7 0.0 0.32" rpy="0 0 0"/>
+	</xacro:sensor_imu>
 <!--
 	<xacro:sensor_asus_xtion_pro name="xtion_pro" parent="base_link">

Commit message: description: replacing hokuyo utm30 by sick s3000 model

File: robospect_description/robots/robospect.urdf.xacro (robot description, xacro)
@@ -37,10 +37,16 @@
 		<origin xyz="0.0 0.0 0.170" rpy="0 0 0"/>
 	</xacro:sensor_imu>
-	<xacro:sensor_hokuyo_utm30lx name="sick_front" parent="base_link">
+	<!--xacro:sensor_hokuyo_utm30lx name="sick_front" parent="base_link">
 		<origin xyz="1.058 0.0 0.0" rpy="0 0 0"/>
 	</xacro:sensor_hokuyo_utm30lx>
 	<xacro:sensor_hokuyo_utm30lx name="sick_rear" parent="base_link">
 		<origin xyz="-1.058 0.0 0.0" rpy="0 0 ${PI}"/>
-	</xacro:sensor_hokuyo_utm30lx>
+	</xacro:sensor_hokuyo_utm30lx!-->
+	<xacro:sensor_sick_s3000 name="sick_front" parent="base_link">
+		<origin xyz="1.058 0.0 0.0" rpy="0 0 0"/>
+	</xacro:sensor_sick_s3000>
+	<xacro:sensor_sick_s3000 name="sick_rear" parent="base_link">
+		<origin xyz="-1.058 0.0 0.0" rpy="0 0 ${PI}"/>
+	</xacro:sensor_sick_s3000>
 <!--
 	<xacro:sensor_hokuyo_urg04lx name="hokuyo1" parent="base_link">
