Commit message: description: Setting new model with real dimensions

File: robospect_description/robots/robospect.urdf.xacro (robot description, xacro)
@@ -73,4 +73,17 @@
 		<origin xyz="0.7 0.0 0.32" rpy="0 0 0"/>
 	</xacro:sensor_imu>
+	<!-- ARM UC3M -->
+    <joint name="arm_joint" type="fixed">
+	  <origin xyz="0.731 0.0 0.308" rpy="0 0 ${-PI/2}"/>
+      <parent link="tip_link"/>
+      <child link="arm_link"/>
+	 </joint>
+	 <link name="arm_link">
+		<inertial>
+			<mass value="1e-5" />
+			<origin xyz="0 0 0" rpy="0 0 0"/>
+			<inertia ixx="1e-6" ixy="0" ixz="0" iyy="1e-6" iyz="0" izz="1e-6" />
+		</inertial>
+	 </link>
 <!--
 	<xacro:sensor_asus_xtion_pro name="xtion_pro" parent="base_link">

File: robospect_description/urdf/bases/robospect_crane.urdf.xacro (robot description, xacro)
@@ -2,10 +2,24 @@
 <robot name="robospect" xmlns:xacro="http://www.ros.org/wiki/xacro">
   <xacro:include filename="$(find robospect_description)/urdf/bases/robospect_crane.gazebo.xacro" />
+  <xacro:property name="joint_1_lower_limit" value="-1.57079"/>
+  <xacro:property name="joint_1_upper_limit" value="1.57079"/>
+  <xacro:property name="joint_2_lower_limit" value="0.0"/>
+  <xacro:property name="joint_2_upper_limit" value="1.824"/>
+  <xacro:property name="joint_3_lower_limit" value="0.0"/>
+  <xacro:property name="joint_3_upper_limit" value="0.5161"/>
+  <xacro:property name="joint_4_lower_limit" value="0.0"/>
+  <xacro:property name="joint_4_upper_limit" value="1.523"/>
+  <xacro:property name="joint_6_lower_limit" value="0.0"/>
+  <xacro:property name="joint_6_upper_limit" value="2.064"/>
+  <xacro:property name="joint_5_lower_limit" value="0.0"/>
+  <xacro:property name="joint_5_upper_limit" value="1.155"/>
+  <xacro:property name="joint_5_pitch" value="1.05"/>
+  <xacro:property name="joint_6_pitch" value="-${joint_6_upper_limit/2.0}"/>
   <xacro:macro name="robospect_crane">
   <!-- FIRST_JOINT -->
     <joint name="crane_first_joint" type="revolute">
       <axis xyz="0 0 1"/>
-      <limit effort="1000.0" lower="-${177.5 * PI / 180}" upper="${177.5 * PI / 180}" velocity="0.5"/>
-      <origin xyz="-0.046851 0 0.3" rpy="0 0 0" />  <!-- height is the clearance -->
+      <limit effort="1000.0" lower="${joint_1_lower_limit}" upper="${joint_1_upper_limit}" velocity="0.5"/>
+      <origin xyz="-0.073 0 0.287" rpy="0 0 0" />  <!-- height is the clearance -->
       <parent link="base_link"/>
       <child link="first_link"/>
@@ -52,6 +66,7 @@
     <joint name="crane_second_joint" type="prismatic">
       <axis xyz="0 0 1"/>
-      <limit effort="1000.0" lower="0.0" upper="2.0" velocity="0.5"/>
-      <origin xyz="-0.28 0 1.25" rpy="0 0 0" />  <!-- height is the clearance -->
+      <limit effort="1000.0" lower="${joint_2_lower_limit}" upper="${joint_2_upper_limit}" velocity="0.5"/>
+      <!--origin xyz="-0.28 0 1.25" rpy="0 0 0" /-->  <!-- height is the clearance -->
+      <origin xyz="-0.305 0 1.442" rpy="0 0 0" />  <!-- height is the clearance -->
       <parent link="first_link"/>
       <child link="second_link"/>
@@ -93,6 +108,6 @@
     <!-- THIRD_JOINT -->
       <joint name="crane_third_joint" type="revolute">
-        <axis xyz="0 1 0"/>
-        <limit effort="100000.0" lower="-1.2" upper="0.06" velocity="0.2"/>
+        <axis xyz="0 -1 0"/>
+        <limit effort="100000.0" lower="${joint_3_lower_limit}" upper="${joint_3_upper_limit}" velocity="0.2"/>
         <origin xyz="0 0 0" rpy="0 0 0" />  <!-- height is the clearance -->
         <parent link="second_link"/>
@@ -136,6 +151,7 @@
       <joint name="crane_fourth_joint" type="prismatic">
         <axis xyz="1 0 0"/>
-        <limit effort="1000.0" lower="0" upper="1.8" velocity="0.5"/>
-        <origin xyz="2.8 0 0.04" rpy="0 0 0" />  <!-- height is the clearance -->
+        <limit effort="1000.0" lower="${joint_4_lower_limit}" upper="${joint_4_upper_limit}" velocity="0.5"/>
+        <!--origin xyz="2.8 0 0.04" rpy="0 0 0" /-->
+        <origin xyz="0.774 0 -0.087" rpy="0 0 0" />  <!-- height is the clearance -->
         <parent link="third_link"/>
         <child link="fourth_link"/>
@@ -175,9 +191,9 @@
       </collision>
     </link>
-    <!-- FIFTH_JOINT -->
+      <!-- FIFTH_JOINT -->
       <joint name="crane_fifth_joint" type="revolute">
         <axis xyz="0 1 0"/>
-        <limit effort="1000.0" lower="-0.7" upper="0.6" velocity="0.5"/>
-        <origin xyz="0 0 0" rpy="0 0 0" />  <!-- height is the clearance -->
+        <limit effort="1000.0" lower="${joint_5_lower_limit}" upper="${joint_5_upper_limit}" velocity="0.5"/>
+        <origin xyz="2.084 0 0.132" rpy="0 ${joint_5_pitch} 0" />
         <parent link="fourth_link"/>
         <child link="fifth_link"/>
@@ -189,6 +205,4 @@
         </joint>
         <actuator name="crane_fifth_joint_act">
-          <!-- This hardwareInterface element exists for compatibility
-               with ROS Hydro. -->
           <hardwareInterface>EffortJointInterface</hardwareInterface>
           <mechanicalReduction>1</mechanicalReduction>
@@ -217,9 +231,9 @@
       </collision>
     </link>
-    <!-- SIXTH_JOINT -->
+     <!-- SIXTH_JOINT -->
       <joint name="crane_sixth_joint" type="revolute">
-        <axis xyz="0 1 0"/>
-        <limit effort="1000.0" lower="-0.5" upper="1.5" velocity="0.5"/>
-        <origin xyz="0.25415 0 0" rpy="0 0 0" />  <!-- height is the clearance -->
+        <axis xyz="0 -1 0"/>
+        <limit effort="1000.0" lower="${joint_6_lower_limit}" upper="${joint_6_upper_limit}" velocity="0.5"/>
+        <origin xyz="0.0 0.0 0.252" rpy="0 -${joint_5_pitch + joint_6_pitch} 0" />  <!-- height is the clearance -->
         <parent link="fifth_link"/>
         <child link="sixth_link"/>
@@ -231,6 +245,4 @@
         </joint>
         <actuator name="crane_sixth_joint_act">
-          <!-- This hardwareInterface element exists for compatibility
-               with ROS Hydro. -->
           <hardwareInterface>EffortJointInterface</hardwareInterface>
           <mechanicalReduction>1</mechanicalReduction>
@@ -244,4 +256,30 @@
         <inertia  ixx="1.391" ixy="0.004"  ixz="0.0"  iyy="6.853"  iyz="0.0"  izz="6.125" />
       </inertial>
+    </link>
+    <!-- SIXTH_AUX_JOINT 1 -->
+    <joint name="crane_sixth_aux_1_joint" type="revolute">
+        <axis xyz="0 -1 0"/>
+        <limit effort="1000.0" lower="${joint_6_lower_limit}" upper="${joint_6_upper_limit}" velocity="0.5"/>
+        <origin xyz="0.0 0.060 0.252" rpy="0 -${joint_5_pitch + joint_6_pitch} 0" />  <!-- height is the clearance -->
+        <parent link="fifth_link"/>
+        <child link="crane_sixth_aux_1_link"/>
+        <mimic joint="crane_sixth_joint"/>
+      </joint>
+      <transmission name="crane_sixth_joint_aux_1_trans">
+        <type>transmission_interface/SimpleTransmission</type>
+        <joint name="crane_sixth_aux_1_joint">
+          <hardwareInterface>EffortJointInterface</hardwareInterface>
+        </joint>
+        <actuator name="crane_sixth_aux_1_joint_act">
+          <hardwareInterface>EffortJointInterface</hardwareInterface>
+          <mechanicalReduction>1</mechanicalReduction>
+        </actuator>
+      </transmission>
+    <link name="crane_sixth_aux_1_link">
+      <inertial>
+        <mass value="1.0" />
+        <origin xyz="0 0 0" />
+        <inertia  ixx="1.391" ixy="0.004"  ixz="0.0"  iyy="6.853"  iyz="0.0"  izz="6.125" />
+      </inertial>
       <visual>
          <origin xyz="0 0 0" rpy="0 0 0" />
@@ -259,52 +297,133 @@
       </collision>
     </link>
-    <!-- SIXTH_AUX_JOINT -->
-      <!--joint name="crane_sixth_aux_joint" type="revolute">
+    <!-- SIXTH_AUX_JOINT 2 -->
+    <joint name="crane_sixth_aux_2_joint" type="revolute">
+        <axis xyz="0 -1 0"/>
+        <limit effort="1000.0" lower="${joint_6_lower_limit}" upper="${joint_6_upper_limit}" velocity="0.5"/>
+        <origin xyz="0.0 -0.060 0.252" rpy="0 -${joint_5_pitch + joint_6_pitch} 0" />  <!-- height is the clearance -->
+        <parent link="fifth_link"/>
+        <child link="crane_sixth_aux_2_link"/>
+        <mimic joint="crane_sixth_joint"/>
+      </joint>
+      <transmission name="crane_sixth_joint_aux_2_trans">
+        <type>transmission_interface/SimpleTransmission</type>
+        <joint name="crane_sixth_aux_2_joint">
+          <hardwareInterface>EffortJointInterface</hardwareInterface>
+        </joint>
+        <actuator name="crane_sixth_aux_2_joint_act">
+          <hardwareInterface>EffortJointInterface</hardwareInterface>
+          <mechanicalReduction>1</mechanicalReduction>
+        </actuator>
+      </transmission>
+    <link name="crane_sixth_aux_2_link">
+      <inertial>
+        <mass value="1.0" />
+        <origin xyz="0 0 0" />
+        <inertia  ixx="1.391" ixy="0.004"  ixz="0.0"  iyy="6.853"  iyz="0.0"  izz="6.125" />
+      </inertial>
+      <visual>
+         <origin xyz="0 0 0" rpy="0 0 0" />
+         <geometry>
+            <mesh filename="package://robospect_description/meshes/bases/robospect_sixth.STL" scale="1 1 1"/>
+         </geometry>
+         <material name="blue">
+         </material>
+      </visual>
+      <collision>
+         <origin xyz="0 0 0" rpy="0 0 0 " />
+         <geometry>
+           <mesh filename="package://robospect_description/meshes/bases/robospect_sixth.STL" scale="1 1 1"/>
+         </geometry>
+      </collision>
+    </link>
+    <!-- SIXTH_AUX_JOINT 3 -->
+    <joint name="crane_sixth_aux_3_joint" type="revolute">
+        <axis xyz="0 -1 0"/>
+        <limit effort="1000.0" lower="${joint_6_lower_limit}" upper="${joint_6_upper_limit}" velocity="0.5"/>
+        <origin xyz="0.264 0.060 0.114" rpy="0 -${joint_5_pitch + joint_6_pitch} 0" />
+        <parent link="fifth_link"/>
+        <child link="crane_sixth_aux_3_link"/>
+        <mimic joint="crane_sixth_joint"/>
+      </joint>
+      <transmission name="crane_sixth_joint_aux_3_trans">
+        <type>transmission_interface/SimpleTransmission</type>
+        <joint name="crane_sixth_aux_3_joint">
+          <hardwareInterface>EffortJointInterface</hardwareInterface>
+        </joint>
+        <actuator name="crane_sixth_aux_3_joint_act">
+          <hardwareInterface>EffortJointInterface</hardwareInterface>
+          <mechanicalReduction>1</mechanicalReduction>
+        </actuator>
+      </transmission>
+    <link name="crane_sixth_aux_3_link">
+      <inertial>
+        <mass value="1.0" />
+        <origin xyz="0 0 0" />
+        <inertia  ixx="1.391" ixy="0.004"  ixz="0.0"  iyy="6.853"  iyz="0.0"  izz="6.125" />
+      </inertial>
+      <visual>
+         <origin xyz="0 0 0" rpy="0 0 0" />
+         <geometry>
+            <mesh filename="package://robospect_description/meshes/bases/robospect_sixth.STL" scale="1 1 1"/>
+         </geometry>
+         <material name="blue">
+         </material>
+      </visual>
+      <collision>
+         <origin xyz="0 0 0" rpy="0 0 0 " />
+         <geometry>
+           <mesh filename="package://robospect_description/meshes/bases/robospect_sixth.STL" scale="1 1 1"/>
+         </geometry>
+      </collision>
+    </link>
+    <!-- SIXTH_AUX_JOINT 4 -->
+    <joint name="crane_sixth_aux_4_joint" type="revolute">
+        <axis xyz="0 -1 0"/>
+        <limit effort="1000.0" lower="${joint_6_lower_limit}" upper="${joint_6_upper_limit}" velocity="0.5"/>
+        <origin xyz="0.264 -0.060 0.114" rpy="0 -${joint_5_pitch + joint_6_pitch} 0" />
+        <parent link="fifth_link"/>
+        <child link="crane_sixth_aux_4_link"/>
+        <mimic joint="crane_sixth_joint"/>
+      </joint>
+      <transmission name="crane_sixth_joint_aux_4_trans">
+        <type>transmission_interface/SimpleTransmission</type>
+        <joint name="crane_sixth_aux_4_joint">
+          <hardwareInterface>EffortJointInterface</hardwareInterface>
+        </joint>
+        <actuator name="crane_sixth_aux_4_joint_act">
+          <hardwareInterface>EffortJointInterface</hardwareInterface>
+          <mechanicalReduction>1</mechanicalReduction>
+        </actuator>
+      </transmission>
+    <link name="crane_sixth_aux_4_link">
+      <inertial>
+        <mass value="1.0" />
+        <origin xyz="0 0 0" />
+        <inertia  ixx="1.391" ixy="0.004"  ixz="0.0"  iyy="6.853"  iyz="0.0"  izz="6.125" />
+      </inertial>
+      <visual>
+         <origin xyz="0 0 0" rpy="0 0 0" />
+         <geometry>
+            <mesh filename="package://robospect_description/meshes/bases/robospect_sixth.STL" scale="1 1 1"/>
+         </geometry>
+         <material name="blue">
+         </material>
+      </visual>
+      <collision>
+         <origin xyz="0 0 0" rpy="0 0 0 " />
+         <geometry>
+           <mesh filename="package://robospect_description/meshes/bases/robospect_sixth.STL" scale="1 1 1"/>
+         </geometry>
+      </collision>
+    </link>
+     <!-- SEVENTH_JOINT -->
+      <joint name="crane_seventh_joint" type="revolute">
         <axis xyz="0 1 0"/>
-        <limit effort="1000.0" lower="0" upper="1.3" velocity="0.5"/>
-        <origin xyz="0.1177 0 -0.26422" rpy="0 0 0" />
-        <parent link="fifth_link"/>
-        <child link="sixth_aux_link"/>
-        <mimic joint="crane_sixth_joint"/>
-      </joint>
-      <transmission name="crane_sixth_aux_joint_trans">
-        <type>transmission_interface/SimpleTransmission</type>
-        <joint name="crane_sixth_aux_joint">
-          <hardwareInterface>EffortJointInterface</hardwareInterface>
-        </joint>
-        <actuator name="crane_sixth_aux_joint_act">
-          <hardwareInterface>EffortJointInterface</hardwareInterface>
-          <mechanicalReduction>1</mechanicalReduction>
-        </actuator>
-      </transmission>
-    <link name="sixth_aux_link">
-      <inertial>
-        <mass value="1.0" />
-        <origin xyz="0 0 0" />
-        <inertia  ixx="1.391" ixy="0.004"  ixz="0.0"  iyy="6.853"  iyz="0.0"  izz="6.125" />
-      </inertial>
-      <visual>
-         <origin xyz="0 0 0" rpy="0 0 0" />
-         <geometry>
-            <mesh filename="package://robospect_description/meshes/bases/robospect_sixth.STL" scale="1 1 1"/>
-         </geometry>
-         <material name="blue">
-         </material>
-      </visual>
-      <collision>
-         <origin xyz="0 0 0" rpy="0 0 0 " />
-         <geometry>
-           <mesh filename="package://robospect_description/meshes/bases/robospect_sixth.STL" scale="1 1 1"/>
-         </geometry>
-      </collision>
-    </link-->
-    <!-- SEVENTH_JOINT -->
-      <joint name="crane_seventh_joint" type="revolute">
-        <axis xyz="0 0 1"/>
-        <limit effort="1000.0" lower="-${90 * PI / 180}" upper="${90 * PI / 180}" velocity="0.5"/>
-        <origin xyz="2.0 0 0" rpy="${90 * PI / 180} 0 0" />  <!-- height is the clearance -->
+        <limit effort="1000.0" lower="-1.57" upper="1.57" velocity="0.5"/>
+        <!--origin xyz="1.239 0 0" rpy="${90 * PI / 180} 0 0" /-->  <!-- height is the clearance -->
+        <origin xyz="1.239 0 0.0" rpy="0 ${joint_6_pitch} 0" />  <!-- height is the clearance -->
         <parent link="sixth_link"/>
         <child link="seventh_link"/>
-        <mimic joint="crane_sixth_joint" offset="-0.485"/>
+        <mimic joint="crane_sixth_joint" multiplier="1.0" offset="0.0"/> <!-- offset="-0.485" -->
       </joint>
       <transmission name="crane_seventh_joint_trans">
@@ -342,9 +461,9 @@
       </collision>
     </link>
-    <!-- TIP_JOINT -->
+        <!-- TIP_JOINT -->
       <joint name="crane_tip_joint" type="revolute">
         <axis xyz="0 0 1"/>
         <limit effort="1000.0" lower="-${90 * PI / 180}" upper="${90 * PI / 180}" velocity="0.5"/>
-        <origin xyz="0.17 -0.15 0.0" rpy="-${90 * PI / 180} 0 0" />  <!-- height is the clearance -->
+        <origin xyz="0.164 0.0 -0.155" rpy="0 0 0" />
         <parent link="seventh_link"/>
         <child link="tip_link"/>

Commit message: description: Moving camera parent link to crane joint 1 link

File: robospect_description/robots/robospect.urdf.xacro (robot description, xacro)
@@ -54,6 +54,6 @@
 	</xacro:sensor_hokuyo_urg04lx>
 -->
-	<xacro:sensor_axis name="camera" parent="base_link">
-		<origin xyz="0.5 0 0.6" rpy="0 ${PI/180} 0"/>
+	<xacro:sensor_axis name="camera" parent="first_link">
+		<origin xyz="0.573 0 0.313" rpy="0 ${PI/180} 0"/>
 	</xacro:sensor_axis>
 	<!-- NAV200 -->

Commit message: description: Moving the location of nav200

File: robospect_description/robots/robospect.urdf.xacro (robot description, xacro)
@@ -37,10 +37,4 @@
 		<origin xyz="0.0 0.0 0.170" rpy="0 0 0"/>
 	</xacro:sensor_imu>
-	<!--xacro:sensor_hokuyo_utm30lx name="sick_front" parent="base_link">
-		<origin xyz="1.058 0.0 0.0" rpy="0 0 0"/>
-	</xacro:sensor_hokuyo_utm30lx>
-	<xacro:sensor_hokuyo_utm30lx name="sick_rear" parent="base_link">
-		<origin xyz="-1.058 0.0 0.0" rpy="0 0 ${PI}"/>
-	</xacro:sensor_hokuyo_utm30lx!-->
 	<xacro:sensor_sick_s3000 name="sick_front" parent="base_link">
 		<origin xyz="1.058 0.0 0.0" rpy="0 0 0"/>
@@ -59,5 +53,6 @@
 	<!-- NAV200 -->
     <joint name="nav200_laser_joint" type="fixed">
-	  <origin xyz="0.9225 0.009 0.408" rpy="0 0 ${-PI/2}"/>
+	  <!--origin xyz="0.9225 0.009 0.408" rpy="0 0 ${-PI/2}"/-->
+	  <origin xyz="0.880 0.0 0.408" rpy="0 0 0"/>
       <parent link="base_link"/>
       <child link="nav200_laser_link"/>

Commit message: description: cleaning code

File: robospect_description/robots/robospect.urdf.xacro (robot description, xacro)
@@ -30,7 +30,4 @@
   <!-- Wheels -->
   <xacro:wheels parent="base_link"/>
-  <!--xacro:front_wheel lr_prefix="right" fr_prefix="rear"/>
-  <xacro:rear_wheel lr_prefix="left" fr_prefix="front">
-  <xacro:rear_wheel lr_prefix="right" fr_prefix="front"/-->
 	<!-- SENSORS -->
 	<xacro:sensor_imu name="imu" parent="base_link">
@@ -43,9 +40,4 @@
 		<origin xyz="-1.058 0.0 0.0" rpy="0 0 ${PI}"/>
 	</xacro:sensor_sick_s3000>
-<!--
-	<xacro:sensor_hokuyo_urg04lx name="hokuyo1" parent="base_link">
-		<origin xyz="-0.1 0.0 0.33" rpy="0 0 0"/>
-	</xacro:sensor_hokuyo_urg04lx>
--->
 	<xacro:sensor_axis name="camera" parent="first_link">
 		<origin xyz="0.573 0 0.313" rpy="0 ${PI/180} 0"/>
@@ -53,5 +45,4 @@
 	<!-- NAV200 -->
     <joint name="nav200_laser_joint" type="fixed">
-	  <!--origin xyz="0.9225 0.009 0.408" rpy="0 0 ${-PI/2}"/-->
 	  <origin xyz="0.880 0.0 0.408" rpy="0 0 0"/>
       <parent link="base_link"/>

File: robospect_description/urdf/bases/robospect_crane.urdf.xacro (robot description, xacro)
@@ -63,5 +63,5 @@
     <material>Gazebo/White</material>
   </gazebo>
-  <!-- SECOND_JOINT -->
+	<!-- SECOND_JOINT -->
     <joint name="crane_second_joint" type="prismatic">
       <axis xyz="0 0 1"/>

Commit message: robospect_description: fixing arm link for the new model

File: robospect_description/robots/robospect.urdf.xacro (robot description, xacro)
@@ -58,10 +58,10 @@
 		</inertial>
 	 </link>
-	<!--xacro:sensor_imu name="imu_crane" parent="tip_link">
-		<origin xyz="0.7 0.0 0.32" rpy="0 0 0"/>
-	</xacro:sensor_imu-->
+	<xacro:sensor_imu name="imu_crane" parent="tip_link">
+		<origin xyz="0.7 0.0 0.153" rpy="0 0 0"/>
+	</xacro:sensor_imu>
 	<!-- ARM UC3M -->
-    <!--joint name="arm_joint" type="fixed">
-	  <origin xyz="0.731 0.0 0.308" rpy="0 0 ${-PI/2}"/>
+    <joint name="arm_joint" type="fixed">
+	  <origin xyz="0.731 0.0 0.153" rpy="0 0 ${-PI/2}"/>
       <parent link="tip_link"/>
       <child link="arm_link"/>
@@ -73,5 +73,5 @@
 			<inertia ixx="1e-6" ixy="0" ixz="0" iyy="1e-6" iyz="0" izz="1e-6" />
 		</inertial>
-	 </link-->
+	 </link>
 <!--
 	<xacro:sensor_asus_xtion_pro name="xtion_pro" parent="base_link">

Commit message: description: Adding new links for the camera system

File: robospect_description/robots/robospect.urdf.xacro (robot description, xacro)
@@ -63,14 +63,31 @@
 	<!-- ARM UC3M -->
     <joint name="arm_joint" type="fixed">
-	  <origin xyz="0.731 0.0 0.153" rpy="0 0 ${-PI/2}"/>
+	  <origin xyz="0.781 0.0 0.153" rpy="0 0 0.0"/>
       <parent link="tip_link"/>
       <child link="arm_link"/>
 	 </joint>
 	 <link name="arm_link">
-		<inertial>
-			<mass value="1e-5" />
-			<origin xyz="0 0 0" rpy="0 0 0"/>
-			<inertia ixx="1e-6" ixy="0" ixz="0" iyy="1e-6" iyz="0" izz="1e-6" />
-		</inertial>
+	 </link>
+	<!-- CAMERA REFERENCE FRAMES -->
+    <joint name="camera_ref_1_joint" type="fixed">
+	  <origin xyz="-0.360 -0.13  0.163" rpy="0 0 0"/>
+      <parent link="arm_link"/>
+      <child link="camera_ref_1_link"/>
+	 </joint>
+	 <link name="camera_ref_1_link">
+	 </link>
+    <joint name="camera_ref_2_joint" type="fixed">
+	  <origin xyz="-0.446 -0.13  0.163" rpy="0 0 0"/>
+      <parent link="arm_link"/>
+      <child link="camera_ref_2_link"/>
+	 </joint>
+	 <link name="camera_ref_2_link">
+	 </link>
+    <joint name="camera_ref_3_joint" type="fixed">
+	  <origin xyz="-0.446 -0.13 0.283" rpy="0 0 0"/>
+      <parent link="arm_link"/>
+      <child link="camera_ref_3_link"/>
+	 </joint>
+	 <link name="camera_ref_3_link">
 	 </link>
 <!--

File: robospect_description/urdf/bases/robospect_crane.gazebo.xacro (robot description, xacro)
@@ -32,11 +32,11 @@
     <material>Gazebo/SkyBlue</material>
   </gazebo>
+  <gazebo reference="fourth_base_link">
+    <material>Gazebo/SkyBlue</material>
+  </gazebo>
   <gazebo reference="fifth_link">
     <material>Gazebo/SkyBlue</material>
   </gazebo>
   <gazebo reference="sixth_link">
-    <material>Gazebo/SkyBlue</material>
-  </gazebo>
-  <gazebo reference="sixth_aux_link">
     <material>Gazebo/SkyBlue</material>
   </gazebo>

File: robospect_description/urdf/bases/robospect_crane.urdf.xacro (robot description, xacro)
@@ -160,9 +160,9 @@
 	</joint>
 	<link name="fourth_base_link">
-      <inertial>
-        <mass value="0.0" />
-        <origin xyz="0 0 0" />
-        <inertia  ixx="0.0" ixy="0.0"  ixz="0.0"  iyy="0.0"  iyz="0.0"  izz="0.0" />
-      </inertial>
+		<inertial>
+			<mass value="2.0" />
+			<origin xyz="0 0 0"/>
+			<inertia  ixx="1.391" ixy="0.004"  ixz="0.0"  iyy="6.853"  iyz="0.0"  izz="6.125" />
+		</inertial>
 	</link>
 	<joint name="crane_fourth_joint" type="prismatic">

Commit message: robospect_common: adding pa10 model to repository and to robospect model

File: robospect_description/robots/robospect.urdf.xacro (robot description, xacro)
@@ -7,4 +7,5 @@
 	<!-- Import Robospect Base -->
 	<xacro:include filename="$(find robospect_description)/urdf/bases/robospect_base.urdf.xacro" />
+	<xacro:include filename="$(find pa10_description)/urdf/pa10.urdf.xacro" />
 	<!-- Import Robospect Crane -->
 	<xacro:include filename="$(find robospect_description)/urdf/bases/robospect_crane.urdf.xacro" />
@@ -72,4 +73,7 @@
 		</inertial>
 	 </link>
+	 <xacro:mitsubishi_pa10  parent="arm_link">
+		<origin xyz="0.0 0.0 0.0" rpy="0 0 ${PI/2}"/>
+	</xacro:mitsubishi_pa10>
 <!--
 	<xacro:sensor_asus_xtion_pro name="xtion_pro" parent="base_link">
