Commit message: description: adjustments

File: robospect_description/robots/robospect.urdf.xacro (robot description, xacro)
@@ -92,7 +92,7 @@
 	 <link name="camera_ref_3_link">
 	 </link>
-	 <xacro:mitsubishi_pa10  parent="arm_link">
+	 <!--xacro:mitsubishi_pa10  parent="arm_link">
 		<origin xyz="0.0 0.0 0.0" rpy="0 0 ${PI/2}"/>
-	</xacro:mitsubishi_pa10>
+	</xacro:mitsubishi_pa10-->
 <!--
 	<xacro:sensor_asus_xtion_pro name="xtion_pro" parent="base_link">

File: robospect_description/urdf/bases/robospect_crane.urdf.xacro (robot description, xacro)
@@ -7,12 +7,10 @@
   <xacro:property name="joint_2_lower_limit" value="0.0"/>
   <xacro:property name="joint_2_upper_limit" value="1.824"/>
-  <xacro:property name="joint_3_lower_limit" value="0.0"/>
-  <xacro:property name="joint_3_upper_limit" value="0.5161"/>
+  <xacro:property name="joint_3_lower_limit" value="-0.166"/>
+  <xacro:property name="joint_3_upper_limit" value="0.3501"/>
   <xacro:property name="joint_4_lower_limit" value="0.0"/>
   <xacro:property name="joint_4_upper_limit" value="1.523"/>
-  <!--xacro:property name="joint_6_lower_limit" value="0.0"/>
-  <xacro:property name="joint_6_upper_limit" value="2.064"/-->
-  <xacro:property name="joint_6_lower_limit" value="-1.032"/>
-  <xacro:property name="joint_6_upper_limit" value="1.032"/>
+  <xacro:property name="joint_6_lower_limit" value="-1.2397"/>
+  <xacro:property name="joint_6_upper_limit" value="0.8283"/>
   <xacro:property name="joint_5_lower_limit" value="0.0"/>
   <xacro:property name="joint_5_upper_limit" value="1.155"/>
@@ -72,5 +70,5 @@
     <joint name="crane_second_joint" type="prismatic">
       <axis xyz="0 0 1"/>
-      <limit effort="1000.0" lower="${joint_2_lower_limit}" upper="${joint_2_upper_limit}" velocity="0.5"/>
+      <limit effort="50000.0" lower="${joint_2_lower_limit}" upper="${joint_2_upper_limit}" velocity="0.25"/>
       <origin xyz="-0.305 0 1.400" rpy="0 0 0" />
       <parent link="first_link"/>
@@ -92,5 +90,5 @@
   <link name="second_link">
     <inertial>
-      <mass value="2.0" />
+      <mass value="10.0" />
       <origin xyz="0 0 0" />
       <inertia  ixx="1.391" ixy="0.004"  ixz="0.0"  iyy="6.853"  iyz="0.0"  izz="6.125" />
@@ -252,5 +250,5 @@
 	<!-- SIXTH_JOINT -->
       <joint name="crane_sixth_joint" type="revolute">
-        <axis xyz="0 0 1"/>
+        <axis xyz="0 0 -1"/>
         <limit effort="1000.0" lower="${joint_6_lower_limit}" upper="${joint_6_upper_limit}" velocity="0.5"/>
         <!--origin xyz="0.0 0.0 0.252" rpy="0 ${PI/2.0} 0" /-->
@@ -301,5 +299,5 @@
         <parent link="sixth_link"/>
         <child link="seventh_link"/>
-        <mimic joint="crane_sixth_joint" multiplier="-1.0" offset="0.0"/>
+        <mimic joint="crane_sixth_joint" multiplier="1.0" offset="0.0"/>
       </joint>
       <transmission name="crane_seventh_joint_trans">

Commit message: Setting new location for arm link

File: robospect_description/robots/robospect.urdf.xacro (robot description, xacro)
@@ -64,5 +64,5 @@
 	<!-- ARM UC3M -->
     <joint name="arm_joint" type="fixed">
-	  <origin xyz="0.781 0.0 0.153" rpy="0 0 0.0"/>
+	  <origin xyz="0.74933 0.0 0.153" rpy="0 0 0.0"/>
       <parent link="tip_link"/>
       <child link="arm_link"/>
@@ -92,4 +92,25 @@
 	 <link name="camera_ref_3_link">
 	 </link>
+    <joint name="camera_ref_4_joint" type="fixed">
+	  <origin xyz="0.0285 -0.320  0.026" rpy="0 0 0"/>
+      <parent link="arm_link"/>
+      <child link="camera_ref_4_link"/>
+	 </joint>
+	 <link name="camera_ref_4_link">
+	 </link>
+    <joint name="camera_ref_5_joint" type="fixed">
+	  <origin xyz="-0.450 -0.320  0.0286" rpy="0 0 0"/>
+      <parent link="arm_link"/>
+      <child link="camera_ref_5_link"/>
+	 </joint>
+	 <link name="camera_ref_5_link">
+	 </link>
+    <joint name="camera_ref_6_joint" type="fixed">
+	  <origin xyz="-0.510 -0.320 -0.4212" rpy="0 0 0"/>
+      <parent link="arm_link"/>
+      <child link="camera_ref_6_link"/>
+	 </joint>
+	 <link name="camera_ref_6_link">
+	 </link>
 	 <!--xacro:mitsubishi_pa10  parent="arm_link">
 		<origin xyz="0.0 0.0 0.0" rpy="0 0 ${PI/2}"/>

Commit message: Minor changes on moveit config and robot description

File: robospect_description/robots/robospect.urdf.xacro (robot description, xacro)
@@ -14,4 +14,5 @@
 	<!-- Import all available sensors -->
 	<xacro:include filename="$(find robotnik_sensors)/urdf/all_sensors.urdf.xacro" />
+	<xacro:include filename="$(find robospect_description)/urdf/bases/camera_frame_v1.urdf.xacro" />
 	<!-- ***************** -->
 	<!-- Global parameters -->
@@ -70,6 +71,9 @@
 	 <link name="arm_link">
 	 </link>
+	 <xacro:camera_frame name="vision" parent="arm_link">
+		<origin xyz="-0.403 0.006 0.3535" rpy="0 0 1.5707"/>
+	 </xacro:camera_frame>
 	<!-- CAMERA REFERENCE FRAMES -->
-    <joint name="camera_ref_1_joint" type="fixed">
+    <!--joint name="camera_ref_1_joint" type="fixed">
 	  <origin xyz="-0.360 -0.13  0.163" rpy="0 0 0"/>
       <parent link="arm_link"/>
@@ -112,5 +116,5 @@
 	 </joint>
 	 <link name="camera_ref_6_link">
-	 </link>
+	 </link-->
 	 <!--xacro:mitsubishi_pa10  parent="arm_link">
 		<origin xyz="0.0 0.0 0.0" rpy="0 0 ${PI/2}"/>

Commit message: moveit_config and description: adding robot arm pa10

File: robospect_description/robots/robospect.urdf.xacro (robot description, xacro)
@@ -117,7 +117,7 @@
 	 <link name="camera_ref_6_link">
 	 </link-->
-	 <!--xacro:mitsubishi_pa10  parent="arm_link">
-		<origin xyz="0.0 0.0 0.0" rpy="0 0 ${PI/2}"/>
-	</xacro:mitsubishi_pa10-->
+	 <xacro:mitsubishi_pa10  parent="arm_link">
+		<origin xyz="0.0 0.0 0.0" rpy="0 0 0"/>
+	</xacro:mitsubishi_pa10>
 <!--
 	<xacro:sensor_asus_xtion_pro name="xtion_pro" parent="base_link">

Commit message: added pan tilt model

File: robospect_description/robots/robospect.urdf.xacro (robot description, xacro)
@@ -12,4 +12,6 @@
 	<!-- Import Robospect Wheels -->
 	<xacro:include filename="$(find robospect_description)/urdf/wheels/standard_wheel.urdf.xacro" />
+	<!-- Import Robospect PTU -->
+	<xacro:include filename="$(find robospect_description)/urdf/bases/ptu_frame_v1.urdf.xacro" />
 	<!-- Import all available sensors -->
 	<xacro:include filename="$(find robotnik_sensors)/urdf/all_sensors.urdf.xacro" />
@@ -120,4 +122,8 @@
 		<origin xyz="0.0 0.0 0.0" rpy="0 0 0"/>
 	</xacro:mitsubishi_pa10>
+	<!-- Robospect_ptu -->
+	<xacro:robospect_ptu parent="arm_link">
+		<origin xyz="-0.45335 0 0.158" rpy="0 0 0"/>
+	</xacro:robospect_ptu>
 <!--
 	<xacro:sensor_asus_xtion_pro name="xtion_pro" parent="base_link">

Commit message: description: setting new position for the cameras related to the new frame v2

File: robospect_description/robots/robospect.urdf.xacro (robot description, xacro)
@@ -16,5 +16,5 @@
 	<!-- Import all available sensors -->
 	<xacro:include filename="$(find robotnik_sensors)/urdf/all_sensors.urdf.xacro" />
-	<xacro:include filename="$(find robospect_description)/urdf/bases/camera_frame_v1.urdf.xacro" />
+	<xacro:include filename="$(find robospect_description)/urdf/bases/camera_frame_v2.urdf.xacro" />
 	<!-- ***************** -->
 	<!-- Global parameters -->
@@ -73,50 +73,10 @@
 	 <link name="arm_link">
 	 </link>
-	 <xacro:camera_frame name="vision" parent="arm_link">
+	 <!--xacro:camera_frame name="vision" parent="arm_link">
 		<origin xyz="-0.403 0.006 0.3535" rpy="0 0 1.5707"/>
+	 </xacro:camera_frame-->
+	 <xacro:camera_frame name="vision" parent="tilt_link">
+		<origin xyz="0 0 0" rpy="0 0 0"/>
 	 </xacro:camera_frame>
-	<!-- CAMERA REFERENCE FRAMES -->
-    <!--joint name="camera_ref_1_joint" type="fixed">
-	  <origin xyz="-0.360 -0.13  0.163" rpy="0 0 0"/>
-      <parent link="arm_link"/>
-      <child link="camera_ref_1_link"/>
-	 </joint>
-	 <link name="camera_ref_1_link">
-	 </link>
-    <joint name="camera_ref_2_joint" type="fixed">
-	  <origin xyz="-0.446 -0.13  0.163" rpy="0 0 0"/>
-      <parent link="arm_link"/>
-      <child link="camera_ref_2_link"/>
-	 </joint>
-	 <link name="camera_ref_2_link">
-	 </link>
-    <joint name="camera_ref_3_joint" type="fixed">
-	  <origin xyz="-0.446 -0.13 0.283" rpy="0 0 0"/>
-      <parent link="arm_link"/>
-      <child link="camera_ref_3_link"/>
-	 </joint>
-	 <link name="camera_ref_3_link">
-	 </link>
-    <joint name="camera_ref_4_joint" type="fixed">
-	  <origin xyz="0.0285 -0.320  0.026" rpy="0 0 0"/>
-      <parent link="arm_link"/>
-      <child link="camera_ref_4_link"/>
-	 </joint>
-	 <link name="camera_ref_4_link">
-	 </link>
-    <joint name="camera_ref_5_joint" type="fixed">
-	  <origin xyz="-0.450 -0.320  0.0286" rpy="0 0 0"/>
-      <parent link="arm_link"/>
-      <child link="camera_ref_5_link"/>
-	 </joint>
-	 <link name="camera_ref_5_link">
-	 </link>
-    <joint name="camera_ref_6_joint" type="fixed">
-	  <origin xyz="-0.510 -0.320 -0.4212" rpy="0 0 0"/>
-      <parent link="arm_link"/>
-      <child link="camera_ref_6_link"/>
-	 </joint>
-	 <link name="camera_ref_6_link">
-	 </link-->
 	 <xacro:mitsubishi_pa10  parent="arm_link">
 		<origin xyz="0.0 0.0 0.0" rpy="0 0 0"/>

File: robospect_description/urdf/sensors/pointgrey_grasshopper3.urdf.xacro (robot description, xacro)
@@ -1,7 +1,19 @@
 <?xml version="1.0"?>
 <robot name="robospect" xmlns:xacro="http://www.ros.org/wiki/xacro">
+	<property name="camera_length_x" value="0.0575" />
+	<property name="camera_length_y" value="0.044" />
+	<property name="camera_length_z" value="0.029" />
 	<xacro:macro name="pointgrey_grasshopper3" params="name parent *origin">
 	<!-- CAMERA BASE_LINK -->
 	<link name="${name}_camera_base_link">
+		<visual>
+			<origin xyz="0 0 ${camera_length_z/2.0}" rpy="0 0 0" />
+			<geometry>
+				<box size="${camera_length_x} ${camera_length_y} ${camera_length_z}" />
+			</geometry>
+				<material name="Cyan">
+			<color rgba="0 1.0 1.0 1.0"/>
+			</material>
+	  </visual>
 	</link>
 	<joint name="${name}_camera_base_joint" type="fixed">

Commit message: description: minor changes

File: robospect_description/robots/robospect.urdf.xacro (robot description, xacro)
@@ -73,7 +73,4 @@
 	 <link name="arm_link">
 	 </link>
-	 <!--xacro:camera_frame name="vision" parent="arm_link">
-		<origin xyz="-0.403 0.006 0.3535" rpy="0 0 1.5707"/>
-	 </xacro:camera_frame-->
 	 <xacro:camera_frame name="vision" parent="tilt_link">
 		<origin xyz="0 0 0" rpy="0 0 0"/>
@@ -86,17 +83,7 @@
 		<origin xyz="-0.45335 0 0.158" rpy="0 0 0"/>
 	</xacro:robospect_ptu>
-<!--
-	<xacro:sensor_asus_xtion_pro name="xtion_pro" parent="base_link">
-		<origin xyz="0.3 0.0 0.3" rpy="0 0 0"/>
-	</xacro:sensor_asus_xtion_pro>
--->
-<!--
-	<xacro:sensor_kinect name="kinect" parent="base_link">
-		<origin xyz="0.3 0.0 0.16" rpy="0 0 0"/>
-	</xacro:sensor_kinect>
--->
-  <!-- gazebo>
-    <plugin name="gazebo_ros_control" filename="libgazebo_ros_control.so"/>
-  </gazebo -->
-  <!-- ros control plugin -->
+	<!-- TIM 571 -->
+	<xacro:sensor_sick_tim571 prefix="tim571_" parent="arm_link">
+		<origin xyz="0.145 -0.302 -0.195" rpy="${PI} -1.082 0"/>
+	</xacro:sensor_sick_tim571>
 </robot>
