Commit message: pa10_description: adding the frames for end effector switches

File: pa10_description/urdf/pa10.urdf.xacro (robot description, xacro)
@@ -161,4 +161,224 @@
     </inertial>
   </link>
+<link name="frame_1">
+  <visual>
+    <origin xyz = "-0.0 -0.0 0.0" rpy="0 0 0"/>
+    <geometry>
+     <box size=" 0.14 0.1 0.01"/>
+    </geometry>
+     <material name="blue">
+     <color rgba="0.5 0.5 0.8 1"/>
+    </material>
+  </visual>
+  <collision>
+    <origin xyz = "-0.0 -0.0 0.0" rpy="0 0 0"/>
+    <geometry>
+     <box size=" 0.14 0.1 0.01"/>
+    </geometry>
+  </collision>
+    <inertial>
+      <mass value="1" />
+      <origin xyz="0 0 0" rpy="0 0 0"/>
+      <inertia ixx="1" ixy="0" ixz="0" iyy="1" iyz="0" izz="1"/>
+    </inertial>
+</link>
+<link name="frame_2">
+  <visual>
+    <origin xyz = "0.0 0.0 0.0" rpy="0 0 0"/>
+    <geometry>
+     <box size=" 0.01 0.1 0.20"/>
+    </geometry>
+     <material name="blue">
+     <color rgba="0.5 0.5 0.9 1"/>
+    </material>
+  </visual>
+  <collision>
+    <origin xyz = "0.0 0.0 0.0" rpy="0 0 0"/>
+    <geometry>
+     <box size=" 0.01 0.1 0.20"/>
+    </geometry>
+  </collision>
+    <inertial>
+      <mass value="1" />
+      <origin xyz="0 0 0" rpy="0 0 0"/>
+      <inertia ixx="1" ixy="0" ixz="0" iyy="1" iyz="0" izz="1"/>
+    </inertial>
+</link>
+<link name="frame_up">
+  <visual>
+    <origin xyz = "0.0 0.0 0" rpy="0 0 0"/>
+    <geometry>
+     <box size=" 0.01 0.26 0.01"/>
+    </geometry>
+     <material name="blue">
+     <color rgba="0.5 0.5 0.9 1"/>
+    </material>
+  </visual>
+  <collision>
+    <origin xyz = "0.0 0.0 0.0" rpy="0 0 0"/>
+    <geometry>
+     <box size=" 0.01 0.26 0.01"/>
+    </geometry>
+  </collision>
+    <inertial>
+      <mass value="1" />
+      <origin xyz="0 0 0" rpy="0 0 0"/>
+      <inertia ixx="1" ixy="0" ixz="0" iyy="1" iyz="0" izz="1"/>
+    </inertial>
+</link>
+<link name="frame_down">
+  <visual>
+    <origin xyz = "0 0 0" rpy="0 0 0"/>
+    <geometry>
+     <box size=" 0.01 0.26 0.01"/>
+    </geometry>
+     <material name="blue">
+     <color rgba="0.5 0.5 0.9 1"/>
+    </material>
+ </visual>
+  <collision>
+    <origin xyz = "0.0 0.0 0.0" rpy="0 0 0"/>
+    <geometry>
+     <box size=" 0.01 0.26 0.01"/>
+    </geometry>
+  </collision>
+    <inertial>
+      <mass value="1" />
+      <origin xyz="0 0 0" rpy="0 0 0"/>
+      <inertia ixx="1" ixy="0" ixz="0" iyy="1" iyz="0" izz="1"/>
+    </inertial>
+</link>
+<link name="frame_right">
+  <visual>
+    <origin xyz = "0.0 0.0 0.0" rpy="0 0 0"/>
+    <geometry>
+     <box size=" 0.125 0.01 0.01"/>
+    </geometry>
+     <material name="blue">
+     <color rgba="0.5 0.5 0.9 1"/>
+    </material>
+  </visual>
+  <collision>
+    <origin xyz = "0.0 0.0 0.0" rpy="0 0 0"/>
+    <geometry>
+     <box size=" 0.12 0.01 0.01"/>
+    </geometry>
+  </collision>
+  <inertial>
+      <mass value="1" />
+      <origin xyz="0 0 0" rpy="0 0 0"/>
+      <inertia ixx="1" ixy="0" ixz="0" iyy="1" iyz="0" izz="1"/>
+    </inertial>
+</link>
+<link name="frame_left">
+  <visual>
+    <origin xyz = "0.0 0 0.0" rpy="0 0 0"/>
+    <geometry>
+     <box size=" 0.125 0.01 0.01"/>
+    </geometry>
+     <material name="blue">
+     <color rgba="0.5 0.5 0.9 1"/>
+    </material>
+  </visual>
+  <collision>
+    <origin xyz = "0.0 0.0 0.0" rpy="0 0 0"/>
+    <geometry>
+     <box size=" 0.12 0.01 0.01"/>
+    </geometry>
+  </collision>
+  <inertial>
+      <mass value="1" />
+      <origin xyz="0 0 0" rpy="0 0 0"/>
+      <inertia ixx="1" ixy="0" ixz="0" iyy="1" iyz="0" izz="1"/>
+  </inertial>
+</link>
+<link name = "sw1">
+ <visual>
+    <origin xyz = "0.0 0.0 0.0" rpy="0 0 0"/>
+    <geometry>
+     <cylinder length="0.02" radius="0.005"/>
+    </geometry>
+    <material name="red">
+     <color rgba="1 0 0 1"/>
+    </material>
+  </visual>
+  <collision>
+    <origin xyz = "0.0 0.0 0.0" rpy="0 0 0"/>
+    <geometry>
+     <cylinder length="0.02" radius="0.005"/>
+    </geometry>
+  </collision>
+  <inertial>
+      <mass value="1" />
+      <origin xyz="0 0 0" rpy="0 0 0"/>
+      <inertia ixx="1" ixy="0" ixz="0" iyy="1" iyz="0" izz="1" />
+  </inertial>
+</link>
+<link name = "sw2">
+ <visual>
+    <origin xyz = "0.0 0.0 0.0" rpy="0 0 0"/>
+    <geometry>
+     <cylinder length="0.02" radius="0.005"/>
+    </geometry>
+    <material name="orange">
+     <color rgba="1 0.6 0 1"/>
+    </material>
+  </visual>
+  <collision>
+    <origin xyz = "0.0 0.0 0.0" rpy="0 0 0"/>
+    <geometry>
+     <cylinder length="0.02" radius="0.005"/>
+    </geometry>
+  </collision>
+  <inertial>
+     <mass value="1e-5" />
+      <origin xyz="0 0 0" rpy="0 0 0"/>
+      <inertia ixx="1e-6" ixy="0" ixz="0" iyy="1e-6" iyz="0" izz="1e-6" />
+  </inertial>
+</link>
+<link name = "sw3">
+ <visual>
+    <origin xyz = "0.0 0.0 0.0" rpy="0 0 0"/>
+    <geometry>
+     <cylinder length="0.02" radius="0.005"/>
+    </geometry>
+    <material name="blue">
+     <color rgba="0 0 0.8 1"/>
+    </material>
+  </visual>
+  <collision>
+    <origin xyz = "0.0 0.0 0.0" rpy="0 0 0"/>
+    <geometry>
+     <cylinder length="0.02" radius="0.005"/>
+    </geometry>
+  </collision>
+  <inertial>
+     <mass value="1e-5" />
+      <origin xyz="0 0 0" rpy="0 0 0"/>
+      <inertia ixx="1e-6" ixy="0" ixz="0" iyy="1e-6" iyz="0" izz="1e-6" />
+  </inertial>
+</link>
+<link name = "sw4">
+ <visual>
+    <origin xyz = "0.0 0.0 0.0" rpy="0 0 0"/>
+    <geometry>
+     <cylinder length="0.02" radius="0.005"/>
+    </geometry>
+    <material name="green">
+     <color rgba="0 0.8 0 1"/>
+    </material>
+  </visual>
+  <collision>
+    <origin xyz = "0.0 0.0 0.0" rpy="0 0 0"/>
+    <geometry>
+     <cylinder length="0.02" radius="0.005"/>
+    </geometry>
+  </collision>
+  <inertial>
+     <mass value="1e-5" />
+      <origin xyz="0 0 0" rpy="0 0 0"/>
+      <inertia ixx="1e-6" ixy="0" ixz="0" iyy="1e-6" iyz="0" izz="1e-6" />
+  </inertial>
+</link>
  <joint name="S0" type="fixed">
     <parent link="${parent}"/>
@@ -231,5 +451,65 @@
   </joint>
 <!-- ......................................................................................... -->
-  <gazebo reference="link0">
+<joint name="link7_frame_1" type="fixed">
+  <parent link = "link7"/>
+  <child link = "frame_1"/>
+  <origin xyz="0 0 0" rpy="0 0 0"/>
+</joint>
+<!-- ......................................................................................... -->
+<joint name="link7_frame_2" type="fixed">
+  <parent link = "link7"/>
+  <child link = "frame_2"/>
+  <origin xyz="0.07 0 0.106" rpy="0 0 0"/>
+</joint>
+<!-- ......................................................................................... -->
+<joint name="link7_frame_up" type="fixed">
+  <parent link = "link7"/>
+  <child link = "frame_up"/>
+  <origin xyz="0.066 0 0.216" rpy="0 0 0"/>
+</joint>
+<!-- ......................................................................................... -->
+<joint name="link7_frame_down" type="fixed">
+  <parent link = "link7"/>
+  <child link = "frame_down"/>
+  <origin xyz="-0.066 0 0.216" rpy="0 0 0"/>
+</joint>
+<!-- ......................................................................................... -->
+<joint name="link7_frame_right" type="fixed">
+  <parent link = "link7"/>
+  <child link = "frame_right"/>
+  <origin xyz="0.0 0.125 0.216" rpy="0 0 0"/>
+</joint>
+<!-- ......................................................................................... -->
+<joint name="link7_frame_left" type="fixed">
+  <parent link = "link7"/>
+  <child link = "frame_left"/>
+  <origin xyz="0 -0.125 0.216" rpy="0 0 0"/>
+</joint>
+<!-- ......................................................................................... -->
+<joint name = "link7_sw1" type="fixed">
+  <parent link = "link7"/>
+  <child link = "sw1"/>
+  <origin xyz = "-0.066 0.123 0.234" rpy = "0.0 0.0 0.0"/>
+</joint>
+<!-- ......................................................................................... -->
+<joint name = "link7_sw2" type="fixed">
+  <parent link = "link7"/>
+  <child link = "sw2"/>
+  <origin xyz = "-0.064 -0.114 0.234" rpy = "0.0 0.0 0.0"/>
+</joint>
+<!-- ......................................................................................... -->
+<joint name = "link7_sw3" type="fixed">
+  <parent link = "link7"/>
+  <child link = "sw3"/>
+  <origin xyz = "0.064 -0.114 0.234" rpy = "0.0 0.0 0.0"/>
+</joint>
+<!-- ......................................................................................... -->
+<joint name = "link7_sw4" type="fixed">
+  <parent link = "link7"/>
+  <child link = "sw4"/>
+  <origin xyz = "0.066 0.123 0.234" rpy = "0.0 0.0 0.0"/>
+</joint>
+<!-- ......................................................................................... -->
+<gazebo reference="link0">
     <material>Gazebo/Blue</material>
     <gravity>0</gravity>
@@ -296,5 +576,5 @@
     <parent link="link5" />
     <child link="hokuyo_link" />
-    <origin xyz="0.0 0.112 0.43" rpy="-1.570796 -1.570796 0.0" />
+    <origin xyz="0.0 0.124 0.43" rpy="-1.570796 -1.570796 0.0" />
   </joint>
 <!-- Hokuyo sensor URDF-->
